File: KiCad/requena.abanto_projecte_vidres/Etapa_de_comunicacio.kicad_sch (KiCad schematic)
At the start: 8 parts, among them J1 DE9_Pins, J2 DE9_Pins, U3 TJA1051TK-3

Commit message: Millora projecte 1
Parts:
- renumbered C5 to C?, D2 to D?, D1 to D?, J1 to J?, J2 to J?, R2 to R?, R1 to R?, U3 to U?
Changed lines of the file:
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@@
 		(dnp no)
 		(fields_autoplaced yes)
-		(property "Reference" "U3"
+		(property "Reference" "U?"
 			(at 103.7433 38.1 0)
 			(effects
@@
 		)
 		(instances
+			(project "requena.abanto_projecte_vidres"
+				(path "/4006572a-320d-4ed7-bf52-f860e1c069c6/4826ec12-9281-4684-8c79-c090e7861812"
+					(reference "U?")
+					(unit 1)
+				)
+			)
 			(project ""
 				(path "/d8765e5a-9256-413e-b62c-c22ecc98887e"
@@
 		(dnp no)
 		(fields_autoplaced yes)
-		(property "Reference" "D2"
+		(property "Reference" "D?"
 			(at 142.24 52.0699 90)
 			(effects
@@
 		)
 		(instances
+			(project "requena.abanto_projecte_vidres"
+				(path "/4006572a-320d-4ed7-bf52-f860e1c069c6/4826ec12-9281-4684-8c79-c090e7861812"
+					(reference "D?")
+					(unit 1)
+				)
+			)
 			(project "Etapa_de_comunicacio"
 				(path "/d8765e5a-9256-413e-b62c-c22ecc98887e"
@@
 		(dnp no)
 		(fields_autoplaced yes)
-		(property "Reference" "C5"
+		(property "Reference" "C?"
 			(at 127.0063 41.91 90)
 			(effects
@@
 		)
 		(instances
+			(project "requena.abanto_projecte_vidres"
+				(path "/4006572a-320d-4ed7-bf52-f860e1c069c6/4826ec12-9281-4684-8c79-c090e7861812"
+					(reference "C?")
+					(unit 1)
+				)
+			)
 			(project ""
 				(path "/d8765e5a-9256-413e-b62c-c22ecc98887e"
@@
 		(dnp no)
 		(fields_autoplaced yes)
-		(property "Reference" "#PWR02"
+		(property "Reference" "#PWR?"
 			(at 133.35 55.88 0)
 			(effects
@@
 		)
 		(instances
+			(project "requena.abanto_projecte_vidres"
+				(path "/4006572a-320d-4ed7-bf52-f860e1c069c6/4826ec12-9281-4684-8c79-c090e7861812"
+					(reference "#PWR?")
+					(unit 1)
+				)
+			)
 			(project "Etapa_de_comunicacio"
 				(path "/d8765e5a-9256-413e-b62c-c22ecc98887e"
@@
 		(dnp no)
 		(fields_autoplaced yes)
-		(property "Reference" "D1"
+		(property "Reference" "D?"
 			(at 142.24 39.3699 90)
 			(effects
@@
 		)
 		(instances
+			(project "requena.abanto_projecte_vidres"
+				(path "/4006572a-320d-4ed7-bf52-f860e1c069c6/4826ec12-9281-4684-8c79-c090e7861812"
+					(reference "D?")
+					(unit 1)
+				)
+			)
 			(project ""
 				(path "/d8765e5a-9256-413e-b62c-c22ecc98887e"
@@
 		(dnp no)
 		(fields_autoplaced yes)
-		(property "Reference" "#PWR01"
+		(property "Reference" "#PWR?"
 			(at 135.89 77.47 0)
 			(effects
@@
 		)
 		(instances
+			(project "requena.abanto_projecte_vidres"
+				(path "/4006572a-320d-4ed7-bf52-f860e1c069c6/4826ec12-9281-4684-8c79-c090e7861812"
+					(reference "#PWR?")
+					(unit 1)
+				)
+			)
 			(project ""
 				(path "/d8765e5a-9256-413e-b62c-c22ecc98887e"
@@
 		(dnp no)
 		(fields_autoplaced yes)
-		(property "Reference" "#PWR04"
+		(property "Reference" "#PWR?"
 			(at 146.05 54.61 0)
 			(effects
@@
 		)
 		(instances
+			(project "requena.abanto_projecte_vidres"
+				(path "/4006572a-320d-4ed7-bf52-f860e1c069c6/4826ec12-9281-4684-8c79-c090e7861812"
+					(reference "#PWR?")
+					(unit 1)
+				)
+			)
 			(project ""
 				(path "/d8765e5a-9256-413e-b62c-c22ecc98887e"
@@
 		(dnp no)
 		(fields_autoplaced yes)
-		(property "Reference" "J1"
+		(property "Reference" "J?"
 			(at 50.8 46.9899 0)
 			(effects
@@
 		)
 		(instances
+			(project "requena.abanto_projecte_vidres"
+				(path "/4006572a-320d-4ed7-bf52-f860e1c069c6/4826ec12-9281-4684-8c79-c090e7861812"
+					(reference "J?")
+					(unit 1)
+				)
+			)
 			(project ""
 				(path "/d8765e5a-9256-413e-b62c-c22ecc98887e"
@@
 		(dnp no)
 		(fields_autoplaced yes)
-		(property "Reference" "R2"
+		(property "Reference" "R?"
 			(at 124.46 52.0699 0)
 			(effects
@@
 		)
 		(instances
+			(project "requena.abanto_projecte_vidres"
+				(path "/4006572a-320d-4ed7-bf52-f860e1c069c6/4826ec12-9281-4684-8c79-c090e7861812"
+					(reference "R?")
+					(unit 1)
+				)
+			)
 			(project "Etapa_de_comunicacio"
 				(path "/d8765e5a-9256-413e-b62c-c22ecc98887e"
@@
 		(dnp no)
 		(fields_autoplaced yes)
-		(property "Reference" "R1"
+		(property "Reference" "R?"
 			(at 124.46 41.9099 0)
 			(effects
@@
 		)
 		(instances
+			(project "requena.abanto_projecte_vidres"
+				(path "/4006572a-320d-4ed7-bf52-f860e1c069c6/4826ec12-9281-4684-8c79-c090e7861812"
+					(reference "R?")
+					(unit 1)
+				)
+			)
 			(project ""
 				(path "/d8765e5a-9256-413e-b62c-c22ecc98887e"
@@
 		(dnp no)
 		(fields_autoplaced yes)
-		(property "Reference" "J2"
+		(property "Reference" "J?"
 			(at 173.99 54.6099 0)
 			(effects
@@
 		)
 		(instances
+			(project "requena.abanto_projecte_vidres"
+				(path "/4006572a-320d-4ed7-bf52-f860e1c069c6/4826ec12-9281-4684-8c79-c090e7861812"
+					(reference "J?")
+					(unit 1)
+				)
+			)
 			(project "Etapa_de_comunicacio"
 				(path "/d8765e5a-9256-413e-b62c-c22ecc98887e"
@@
 		(dnp no)
 		(fields_autoplaced yes)
-		(property "Reference" "#PWR03"
+		(property "Reference" "#PWR?"
 			(at 46.99 38.1 0)
 			(effects
@@
 		)
 		(instances
+			(project "requena.abanto_projecte_vidres"
+				(path "/4006572a-320d-4ed7-bf52-f860e1c069c6/4826ec12-9281-4684-8c79-c090e7861812"
+					(reference "#PWR?")
+					(unit 1)
+				)
+			)
 			(project ""
 				(path "/d8765e5a-9256-413e-b62c-c22ecc98887e"

Commit message: millora
Parts:
- removed C?: C_Small, symbol Device:C_Small
- removed D? (x2): D, symbol Device:D
- removed J? (x2): DE9_Pins, symbol Connector:DE9_Pins
- removed R? (x2): R, symbol Device:R
- removed U?: TJA1051TK-3, Package_SON:HVSON-8-1EP_3x3mm_P0.65mm_EP1.6x2.4mm, symbol Interface_CAN_LIN:TJA1051TK-3
Connections:
- no-connect marks 11 -> 0
Other:
- note removed: "CAN"
- note removed: "TTL-232R"
- note removed: "USART"
