File: KiCad/requena.abanto_projecte_vidres/Etapa_de_alimentacio.kicad_sch (KiCad schematic)
At the start: 0 parts

Commit message: etapa alimentación empezada
Parts:
- added U1: TSR2-2450, Converter_DCDC:Converter_DCDC_TRACO_TSR2-xxxx_THT, symbol Converter_DCDC:TSR2-2450
- added U2: LM1117DT-3.3, Package_TO_SOT_SMD:TO-252-3_TabPin2, symbol Regulator_Linear:LM1117DT-3.3
Connections:
- new net +12V: U1.1 (Vin)
- new net GND: U1.2 (GND), U2.1 (GND)
- new net VCC: U2.2 (VO)
- new net V_OUT_DCDC: U1.3 (Vout), U2.3 (VI)

Commit message: proteccion alimentacion
Parts:
- added C1, C3: 1uF, symbol Device:C_Polarized
- added C2, C4: 100nF, symbol Device:C
- added D1: D, symbol Device:D
- added D2: D_Zener, symbol Device:D_Zener
Connections:
- net +12V: now also D1.2 (A); no longer U1.1 (Vin)
- net GND: now also C1.2, C2.2, C3.2, C4.2, D2.2 (A)
- net VCC: now also C2.1, C3.1
- new net: C1.1, C4.1, D1.1 (K), D2.1 (K), U1.1 (Vin)
Other:
- moved on the sheet: U1, U2

Commit message: Millora projecte 1
Parts:
- removed C1, C3: 1uF, symbol Device:C_Polarized
- removed C2, C4: 100nF, symbol Device:C
- removed D1: D, symbol Device:D
- removed D2: D_Zener, symbol Device:D_Zener
- removed U1: TSR2-2450, Converter_DCDC:Converter_DCDC_TRACO_TSR2-xxxx_THT, symbol Converter_DCDC:TSR2-2450
- removed U2: LM1117DT-3.3, Package_TO_SOT_SMD:TO-252-3_TabPin2, symbol Regulator_Linear:LM1117DT-3.3
