File: KiCad/requena.abanto_projecte_vidres/Etapa_de_processament.kicad_sch (KiCad schematic)
At the start: 45 parts

Commit message: correcions
Parts:
- gave numbers to parts that had none: 45

Commit message: millora_petjades
Parts:
- C10, C11, C12, C18, C19, C20, C21, C22, C7, C8, C9: footprint (none) -> Capacitor_SMD:C_1206_3216Metric
- C13, C15: value C -> 22 pF; footprint (none) -> Capacitor_SMD:C_0805_2012Metric
- C14, C16, C17: footprint (none) -> Capacitor_SMD:C_0805_2012Metric
- D3, D4: footprint (none) -> Diode_SMD:D_0805_2012Metric
- J1: footprint (none) -> TerminalBlock:TerminalBlock_Xinya_XY308-2.54-5P_1x05_P2.54mm_Horizontal
- J2: footprint (none) -> Connector_JST:JST_XH_B4B-XH-AM_1x04_P2.50mm_Vertical
- J3, J4: footprint (none) -> Connector_Dsub:DSUB-9_Pins_Vertical_P2.77x2.84mm
- JP1: footprint (none) -> Connector_PinHeader_2.54mm:PinHeader_1x03_P2.54mm_Horizontal
- R10, R11, R12, R13, R4, R5, R7, R8, R9: footprint (none) -> Resistor_SMD:R_1206_3216Metric
- R6: value R -> 10k; footprint (none) -> Resistor_SMD:R_1206_3216Metric
- SW1: footprint (none) -> Button_Switch_SMD:SW_SPDT_PCM12
- SW2: footprint (none) -> Button_Switch_SMD:SW_Push_1P1T_NO_E-Switch_TL3301NxxxxxG
- SW3, SW4, SW5, SW6: footprint (none) -> Button_Switch_SMD:SW_SPST_Omron_B3FS-100xP
- Y1: value Crystal -> 27.12 MHz; footprint (none) -> Crystal:Crystal_SMD_HC49-SD
- Y2: value Crystal -> 8 MHz; footprint (none) -> Crystal:Crystal_SMD_HC49-SD
Other:
- moved on the sheet: C18

Commit message: milora_esquema_i_layoutcomençat
Connections:
- net CLOSED_FC: no longer U10.2 (Y6)
- net GND: no longer JP1.2 (C), U8.1 (~{MCLR})
- net OPEN_FC: no longer U10.4 (Y7)
- new net: JP1.2 (C), U8.1 (~{MCLR})
- no-connect marks 20 -> 22
Other:
- moved on the sheet: JP1, R6, SW2
Changed lines of the file:
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@@
 	)
 	(junction
-		(at 106.68 74.93)
-		(diameter 0)
-		(color 0 0 0 0)
-	)
-	(junction
-		(at 106.68 86.36)
+		(at 107.95 73.66)
 		(diameter 0)
 		(color 0 0 0 0)
@@
 	)
 	(junction
+		(at 107.95 88.9)
+		(diameter 0)
+		(color 0 0 0 0)
+	)
+	(junction
 		(at 83.82 22.86)
 		(diameter 0)
@@
 		(color 0 0 0 0)
 	)
-	(junction
-		(at 106.68 88.9)
-		(diameter 0)
-		(color 0 0 0 0)
+	(no_connect
+		(at 241.3 95.25)
 	)
 	(no_connect
@@
 	)
 	(no_connect
+		(at 241.3 97.79)
+	)
+	(no_connect
 		(at 55.88 170.18)
 	)
@@
 	(wire
 		(pts
-			(xy 104.14 74.93) (xy 106.68 74.93)
-		)
-		(stroke
-			(width 0)
-			(type default)
-		)
-	)
-	(wire
-		(pts
 			(xy 68.58 180.34) (xy 68.58 187.96)
 		)
@@
 	(wire
 		(pts
-			(xy 97.79 78.74) (xy 97.79 86.36)
+			(xy 97.79 77.47) (xy 97.79 86.36)
 		)
 		(stroke
@@
 	(wire
 		(pts
-			(xy 97.79 86.36) (xy 106.68 86.36)
+			(xy 97.79 86.36) (xy 132.08 86.36)
 		)
 		(stroke
@@
 	(wire
 		(pts
+			(xy 104.14 73.66) (xy 107.95 73.66)
+		)
+		(stroke
+			(width 0)
+			(type default)
+		)
+	)
+	(wire
+		(pts
 			(xy 176.53 36.83) (xy 207.01 36.83)
 		)
@@
 	(wire
 		(pts
-			(xy 106.68 73.66) (xy 106.68 74.93)
+			(xy 107.95 72.39) (xy 107.95 73.66)
 		)
 		(stroke
@@
 	(wire
 		(pts
-			(xy 130.81 88.9) (xy 106.68 88.9)
-		)
-		(stroke
-			(width 0)
-			(type default)
-		)
-	)
-	(wire
-		(pts
 			(xy 76.2 180.34) (xy 76.2 187.96)
 		)
@@
 	(wire
 		(pts
+			(xy 107.95 85.09) (xy 107.95 88.9)
+		)
+		(stroke
+			(width 0)
+			(type default)
+		)
+	)
+	(wire
+		(pts
 			(xy 95.25 39.37) (xy 99.06 39.37)
 		)
@@
 	(wire
 		(pts
-			(xy 106.68 74.93) (xy 106.68 76.2)
+			(xy 107.95 73.66) (xy 107.95 74.93)
 		)
 		(stroke
@@
 	(wire
 		(pts
-			(xy 91.44 74.93) (xy 91.44 93.98)
-		)
-		(stroke
-			(width 0)
-			(type default)
-		)
-	)
-	(wire
-		(pts
-			(xy 233.68 95.25) (xy 241.3 95.25)
+			(xy 91.44 73.66) (xy 91.44 93.98)
 		)
 		(stroke
@@
 	(wire
 		(pts
-			(xy 233.68 97.79) (xy 241.3 97.79)
-		)
-		(stroke
-			(width 0)
-			(type default)
-		)
-	)
-	(wire
-		(pts
 			(xy 144.78 120.65) (xy 142.24 120.65)
 		)
@@
 	(wire
 		(pts
-			(xy 106.68 86.36) (xy 106.68 88.9)
-		)
-		(stroke
-			(width 0)
-			(type default)
-		)
-	)
-	(wire
-		(pts
 			(xy 91.44 157.48) (xy 96.52 157.48)
 		)
@@
 	(wire
 		(pts
-			(xy 106.68 86.36) (xy 132.08 86.36)
-		)
-		(stroke
-			(width 0)
-			(type default)
-		)
-	)
-	(wire
-		(pts
 			(xy 24.13 128.27) (xy 34.29 128.27)
 		)
@@
 	(wire
 		(pts
-			(xy 106.68 63.5) (xy 106.68 66.04)
+			(xy 107.95 62.23) (xy 107.95 64.77)
 		)
 		(stroke
@@
 	(wire
 		(pts
+			(xy 107.95 88.9) (xy 130.81 88.9)
+		)
+		(stroke
+			(width 0)
+			(type default)
+		)
+	)
+	(wire
+		(pts
 			(xy 194.31 40.64) (xy 194.31 35.56)
 		)
@@
 	(wire
 		(pts
-			(xy 81.28 88.9) (xy 106.68 88.9)
+			(xy 81.28 88.9) (xy 107.95 88.9)
 		)
 		(stroke
@@
 	(global_label "VCC"
 		(shape input)
-		(at 106.68 63.5 90)
+		(at 107.95 62.23 90)
 		(fields_autoplaced yes)
 		(effects
@@
 		)
 		(property "Intersheetrefs" "${INTERSHEET_REFS}"
-			(at 106.68 56.8862 90)
+			(at 107.95 55.6162 90)
 			(effects
 				(font
@@
 		)
 	)
-	(global_label "OPEN_FC"
-		(shape input)
-		(at 233.68 97.79 180)
-		(fields_autoplaced yes)
-		(effects
-			(font
-				(size 1.27 1.27)
-			)
-			(justify right)
-		)
-		(property "Intersheetrefs" "${INTERSHEET_REFS}"
-			(at 222.2886 97.79 0)
-			(effects
-				(font
-					(size 1.27 1.27)
-				)
-				(justify right)
-				(hide yes)
-			)
-		)
-	)
 	(global_label "VCC"
 		(shape input)
@@
 		)
 	)
-	(global_label "CLOSED_FC"
-		(shape input)
-		(at 233.68 95.25 180)
-		(fields_autoplaced yes)
-		(effects
-			(font
-				(size 1.27 1.27)
-			)
-			(justify right)
-		)
-		(property "Intersheetrefs" "${INTERSHEET_REFS}"
-			(at 220.1115 95.25 0)
-			(effects
-				(font
-					(size 1.27 1.27)
-				)
-				(justify right)
-				(hide yes)
-			)
-		)
-	)
 	(symbol
 		(lib_id "Interface_CAN_LIN:TJA1051TK-3")
@@
 	(symbol
 		(lib_id "Switch:SW_Push")
-		(at 106.68 81.28 270)
+		(at 107.95 80.01 270)
 		(unit 1)
 		(exclude_from_sim no)
@@
 		(fields_autoplaced yes)
 		(property "Reference" "SW2"
-			(at 110.49 80.0099 90)
+			(at 111.76 78.7399 90)
 			(effects
 				(font
@@
 		)
 		(property "Value" "SW_Push"
-			(at 110.49 82.5499 90)
+			(at 111.76 81.2799 90)
 			(effects
 				(font
@@
 		)
 		(property "Footprint" "Button_Switch_SMD:SW_Push_1P1T_NO_E-Switch_TL3301NxxxxxG"
-			(at 111.76 81.28 0)
+			(at 113.03 80.01 0)
 			(effects
 				(font
@@
 		)
 		(property "Datasheet" "~"
-			(at 111.76 81.28 0)
+			(at 113.03 80.01 0)
 			(effects
 				(font
@@
 		)
 		(property "Description" "Push button switch, generic, two pins"
-			(at 106.68 81.28 0)
+			(at 107.95 80.01 0)
 			(effects
 				(font
@@
 	(symbol
 		(lib_id "Device:R")
-		(at 106.68 69.85 180)
+		(at 107.95 68.58 180)
 		(unit 1)
 		(exclude_from_sim no)
@@
 		(fields_autoplaced yes)
 		(property "Reference" "R6"
-			(at 109.22 68.5799 0)
+			(at 110.49 67.3099 0)
 			(effects
 				(font
@@
 		)
 		(property "Value" "10k"
-			(at 109.22 71.1199 0)
+			(at 110.49 69.8499 0)
 			(effects
 				(font
@@
 		)
 		(property "Footprint" "Resistor_SMD:R_1206_3216Metric"
-			(at 108.458 69.85 90)
+			(at 109.728 68.58 90)
 			(effects
 				(font
@@
 		)
 		(property "Datasheet" "~"
-			(at 106.68 69.85 0)
+			(at 107.95 68.58 0)
 			(effects
 				(font
@@
 		)
 		(property "Description" "Resistor"
-			(at 106.68 69.85 0)
+			(at 107.95 68.58 0)
 			(effects
 				(font
@@
 	(symbol
 		(lib_id "Jumper:Jumper_3_Open")
-		(at 97.79 74.93 0)
+		(at 97.79 73.66 0)
 		(unit 1)
 		(exclude_from_sim no)
@@
 		(fields_autoplaced yes)
 		(property "Reference" "JP1"
-			(at 97.79 68.58 0)
+			(at 97.79 67.31 0)
 			(effects
 				(font
@@
 		)
 		(property "Value" "Jumper_3_Open"
-			(at 97.79 71.12 0)
+			(at 97.79 69.85 0)
 			(effects
 				(font
@@
 		)
 		(property "Footprint" "Connector_PinHeader_2.54mm:PinHeader_1x03_P2.54mm_Horizontal"
-			(at 97.79 74.93 0)
+			(at 97.79 73.66 0)
 			(effects
 				(font
@@
 		)
 		(property "Datasheet" "~"
-			(at 97.79 74.93 0)
+			(at 97.79 73.66 0)
 			(effects
 				(font
@@
 		)
 		(property "Description" "Jumper, 3-pole, both open"
-			(at 97.79 74.93 0)
+			(at 97.79 73.66 0)
 			(effects
 				(font

Commit message: :(
Other:
- company: (none) -> AUTORS: ÀLEX REQUENA i ALFRED ABANTO
- title: (none) -> ETAPA DE PROCESSAMENT
Changed lines of the file:
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@@
 	(generator_version "9.0")
 	(paper "A4")
+	(title_block
+		(title "ETAPA DE PROCESSAMENT")
+		(company "AUTORS: ÀLEX REQUENA i ALFRED ABANTO")
+	)
 	(text "CAN"
 		(exclude_from_sim no)

Commit message: Millora del micro a 44 pins
Parts:
- removed C22: 100n, Capacitor_SMD:C_1206_3216Metric, symbol Device:C
- removed U10: NMUX1308PW, Package_SO:TSSOP-16_4.4x5mm_P0.65mm, symbol Analog_Switch:NMUX1308PW
- removed U8: PIC24HJ128GP502, Package_SO:SSOP-28_5.3x10.2mm_P0.65mm, symbol biblioteca_de_projecte:PIC18F23K20_ISS
- added U6: PIC24HJ128GP502, Package_QFP:TQFP-44_10x10mm_P0.8mm, symbol MCU_Microchip_PIC32:PIC32MX250F128D-IPT
- Y1, Y2: footprint Crystal:Crystal_SMD_HC49-SD -> Crystal:Crystal_SMD_3225-4Pin_3.2x2.5mm
Connections:
- net AN0: now also U6.19 (RA0/ANO)
- net GND: no longer C14.2, C16.2, C18.2, C19.2, J1.3 (Pin_3), J3.5, SW2.2
- net OSC1: now also U6.31 (OSC2)
- net OSC2: now also U6.30 (OSC1)
- net at C17.1: now also U6.7 (VCAP)
- new net: C14.2, C16.2
- new net: C18.2, C19.2, J3.5
- new net: U6.28 (VDD), U6.40 (VDD)
- new net: U6.29 (VSS), U6.39 (VSS), U6.6 (VSS)
- new net: J1.3 (Pin_3), SW2.2
- no-connect marks 22 -> 18
Other:
- note removed: "MUX 8-1"
- moved on the sheet: C10, C11, C12, C13, C14, C15, C16, C17, C7, C8, C9, J2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

Commit message: .
Connections:
- net CAN_RX: now also U6.22 (RB1/RP1)
- net CAN_TX: now also U6.21 (RB0/RP0)
- net CLOSED_FC: now also U6.4 (RC8)
- net CLOSE_D: now also U6.37 (RC4)
- net DOWN_W: now also U6.2 (RC6)
- net GND: now also C14.2, C16.2, C18.1, C19.2, J1.3 (Pin_3), J3.5, SW2.2, U6.16 (AVSS), U6.29 (VSS), U6.39 (VSS), U6.6 (VSS)
- net OPEN_D: now also U6.38 (RC5)
- net OPEN_FC: now also U6.5 (RC9)
- net PGEC1: now also U6.36 (RC3)
- net PGED1: now also U6.27 (RC2)
- net PWM: now also U6.33 (RB4)
- net RB15: now also U6.41 (RB5)
- net UART_RX: now also U6.24 (RB3)
- net UART_TX: now also U6.23 (RB2)
- net UP_W: now also U6.3 (RC7)
- net VCC: now also C18.2, U6.17 (AVDD), U6.28 (VDD), U6.40 (VDD); no longer C18.1
- net at U6.18 (~{MCLR}): now also JP1.2 (C)
Other:
- moved on the sheet: C14, C16, C17, C18, J1, J3, JP1, R6, SW2, U6, Y2

Commit message: esquema acabat
Parts:
- removed J2: Conn_01x04_Socket, Connector_JST:JST_XH_B4B-XH-AM_1x04_P2.50mm_Vertical, symbol Connector:Conn_01x04_Socket
- added J6: Conn_01x04, TerminalBlock:TerminalBlock_Xinya_XY308-2.54-4P_1x04_P2.54mm_Horizontal, symbol Connector_Generic:Conn_01x04
- J3, J4: footprint Connector_Dsub:DSUB-9_Pins_Vertical_P2.77x2.84mm -> Connector_Dsub:DSUB-9_Pins_Horizontal_P2.77x2.84mm_EdgePinOffset4.94mm_Housed_MountingHolesOffset4.94mm
- Y1, Y2: footprint Crystal:Crystal_SMD_3225-4Pin_3.2x2.5mm -> Crystal:Crystal_SMD_3215-2Pin_3.2x1.5mm
Connections:
- net INA: now also U6.13 (RA7)
- net INB: now also U6.32 (RA8)
- net IRQ: now also U6.1 (RB9)
- net MISO: now also U6.44 (RB8)
- net MOSI: now also U6.8 (RB10)
- net NRSTPD: now also U6.43 (RB7)
- net SCK: now also U6.9 (RB11)
- net at U7.19 (AUX1): now also J6.3 (Pin_3)
- net at U7.20 (AUX2): now also J6.4 (Pin_4)
- net at U7.7 (SIGIN): now also J6.1 (Pin_1)
- net at U7.8 (SIGOUT): now also J6.2 (Pin_2)
- no-connect marks 18 -> 29
Other:
- moved on the sheet: C10, C11, C12, C13, C14, C15, C16, C17, C18, C19, C20, C21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

Commit message: a mimir
Parts:
- J1: footprint TerminalBlock:TerminalBlock_Xinya_XY308-2.54-5P_1x05_P2.54mm_Horizontal -> Connector_PinHeader_2.54mm:PinHeader_1x05_P2.54mm_Vertical
- J6: footprint TerminalBlock:TerminalBlock_Xinya_XY308-2.54-4P_1x04_P2.54mm_Horizontal -> Connector_PinHeader_2.54mm:PinHeader_1x05_P2.54mm_Vertical
- JP1: footprint Connector_PinHeader_2.54mm:PinHeader_1x03_P2.54mm_Horizontal -> Connector_PinHeader_2.54mm:PinHeader_1x03_P2.54mm_Vertical
Connections:
- net PGEC1: now also U6.26 (RC1); no longer U6.36 (RC3)
- net UART_RX: now also U6.10 (RB12); no longer U6.24 (RB3)
- net UART_TX: now also U6.11 (RB13); no longer U6.23 (RB2)
Changed lines of the file:
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@@
 	)
 	(junction
-		(at 111.76 76.2)
-		(diameter 0)
-		(color 0 0 0 0)
-	)
-	(junction
 		(at 30.48 129.54)
 		(diameter 0)
@@
 	)
 	(junction
-		(at 203.2 101.6)
-		(diameter 0)
-		(color 0 0 0 0)
-	)
-	(junction
 		(at 111.76 181.61)
 		(diameter 0)
@@
 	)
 	(junction
+		(at 111.76 76.2)
+		(diameter 0)
+		(color 0 0 0 0)
+	)
+	(junction
 		(at 157.48 129.54)
 		(diameter 0)
@@
 	)
 	(no_connect
-		(at 52.07 176.53)
+		(at 180.34 106.68)
 	)
 	(no_connect
-		(at 101.6 86.36)
+		(at 52.07 176.53)
 	)
 	(no_connect
-		(at 138.43 106.68)
+		(at 101.6 86.36)
 	)
 	(no_connect
@@
 	)
 	(no_connect
-		(at 101.6 68.58)
+		(at 138.43 78.74)
 	)
 	(no_connect
-		(at 138.43 114.3)
+		(at 101.6 68.58)
 	)
 	(no_connect
@@
 	)
 	(no_connect
-		(at 138.43 104.14)
-	)
-	(no_connect
 		(at 180.34 81.28)
 	)
@@
 	)
 	(no_connect
-		(at 180.34 101.6)
-	)
-	(no_connect
 		(at 180.34 99.06)
 	)
@@
 	)
 	(no_connect
+		(at 138.43 106.68)
+	)
+	(no_connect
 		(at 101.6 71.12)
 	)
@@
 		(at 180.34 73.66)
 	)
+	(no_connect
+		(at 138.43 76.2)
+	)
 	(wire
 		(pts
@@
 	(wire
 		(pts
+			(xy 135.89 104.14) (xy 138.43 104.14)
+		)
+		(stroke
+			(width 0)
+			(type default)
+		)
+	)
+	(wire
+		(pts
 			(xy 35.56 52.07) (xy 35.56 55.88)
 		)
@@
 	(wire
 		(pts
+			(xy 137.16 78.74) (xy 137.16 114.3)
+		)
+		(stroke
+			(width 0)
+			(type default)
+		)
+	)
+	(wire
+		(pts
 			(xy 234.95 129.54) (xy 251.46 129.54)
 		)
@@
 	(wire
 		(pts
+			(xy 111.76 76.2) (xy 135.89 76.2)
+		)
+		(stroke
+			(width 0)
+			(type default)
+		)
+	)
+	(wire
+		(pts
 			(xy 121.92 129.54) (xy 134.62 129.54)
 		)
@@
 	(wire
 		(pts
+			(xy 107.95 78.74) (xy 137.16 78.74)
+		)
+		(stroke
+			(width 0)
+			(type default)
+		)
+	)
+	(wire
+		(pts
 			(xy 180.34 40.64) (xy 181.61 40.64)
 		)
@@
 	(wire
 		(pts
+			(xy 135.89 76.2) (xy 135.89 104.14)
+		)
+		(stroke
+			(width 0)
+			(type default)
+		)
+	)
+	(wire
+		(pts
 			(xy 148.59 66.04) (xy 175.26 66.04)
 		)
@@
 	(wire
 		(pts
-			(xy 138.43 76.2) (xy 111.76 76.2)
-		)
-		(stroke
-			(width 0)
-			(type default)
-		)
-	)
-	(wire
-		(pts
 			(xy 133.35 91.44) (xy 138.43 91.44)
 		)
@@
 	(wire
 		(pts
-			(xy 138.43 78.74) (xy 107.95 78.74)
-		)
-		(stroke
-			(width 0)
-			(type default)
-		)
-	)
-	(wire
-		(pts
 			(xy 257.81 68.58) (xy 257.81 80.01)
 		)
@@
 	(wire
 		(pts
-			(xy 203.2 101.6) (xy 205.74 101.6)
+			(xy 20.32 129.54) (xy 30.48 129.54)
 		)
 		(stroke
@@
 	(wire
 		(pts
-			(xy 20.32 129.54) (xy 30.48 129.54)
+			(xy 180.34 104.14) (xy 181.61 104.14)
 		)
 		(stroke
@@
 	(wire
 		(pts
-			(xy 180.34 104.14) (xy 181.61 104.14)
-		)
-		(stroke
-			(width 0)
-			(type default)
-		)
-	)
-	(wire
-		(pts
 			(xy 111.76 160.02) (xy 121.92 160.02)
 		)
@@
 	(wire
 		(pts
-			(xy 180.34 106.68) (xy 181.61 106.68)
+			(xy 180.34 101.6) (xy 181.61 101.6)
 		)
 		(stroke
@@
 		)
 	)
+	(wire
+		(pts
+			(xy 137.16 114.3) (xy 138.43 114.3)
+		)
+		(stroke
+			(width 0)
+			(type default)
+		)
+	)
 	(global_label "NRSTPD"
 		(shape input)
@@
 	(global_label "PGEC1"
 		(shape input)
-		(at 181.61 106.68 0)
+		(at 181.61 101.6 0)
 		(fields_autoplaced yes)
 		(effects
@@
 		)
 		(property "Intersheetrefs" "${INTERSHEET_REFS}"
-			(at 190.7637 106.68 0)
+			(at 190.7637 101.6 0)
 			(effects
 				(font
@@
 			)
 		)
-		(property "Footprint" "TerminalBlock:TerminalBlock_Xinya_XY308-2.54-4P_1x04_P2.54mm_Horizontal"
+		(property "Footprint" "Connector_PinHeader_2.54mm:PinHeader_1x05_P2.54mm_Vertical"
 			(at 127 154.94 0)
 			(effects
@@
 			)
 		)
-		(property "Footprint" "TerminalBlock:TerminalBlock_Xinya_XY308-2.54-5P_1x05_P2.54mm_Horizontal"
+		(property "Footprint" "Connector_PinHeader_2.54mm:PinHeader_1x05_P2.54mm_Vertical"
 			(at 91.44 119.38 0)
 			(effects
@@
 			)
 		)
-		(property "Footprint" "Connector_PinHeader_2.54mm:PinHeader_1x03_P2.54mm_Horizontal"
+		(property "Footprint" "Connector_PinHeader_2.54mm:PinHeader_1x03_P2.54mm_Vertical"
 			(at 111.76 104.14 0)
 			(effects
