File: KiCad/requena.abanto_projecte_vidres/Etapa_de_processament.kicad_sch (KiCad schematic)
At the start: 43 parts, among them J1 Conn_01x05, J3 DE9_Pins, J4 DE9_Pins, J6 Conn_01x04, SW1 SW_Push_SPDT, SW2 SW_Push, SW3 SW_Omron_B3FS, SW4 SW_Omron_B3FS, SW5 SW_Omron_B3FS, SW6 SW_Omron_B3FS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

Commit message: primera pcb
Parts:
- J6: footprint Connector_PinHeader_2.54mm:PinHeader_1x05_P2.54mm_Vertical -> Connector_PinHeader_2.54mm:PinHeader_1x04_P2.54mm_Vertical
Connections:
- net CAN_RX: now also U6.21 (RB0/RP0); no longer U6.22 (RB1/RP1)
- net CAN_TX: now also U6.22 (RB1/RP1); no longer U6.21 (RB0/RP0)
- net CLOSE_D: now also U6.9 (RB11); no longer U6.37 (RC4)
- net IRQ: now also U6.36 (RC3); no longer U6.1 (RB9)
- net MISO: now also U6.43 (RB7); no longer U6.44 (RB8)
- net MOSI: now also U6.38 (RC5); no longer U6.8 (RB10)
- net NRSTPD: now also U6.41 (RB5); no longer U6.43 (RB7)
- net OPEN_D: now also U6.8 (RB10); no longer U6.38 (RC5)
- net PGEC1: now also J1.4 (Pin_4); no longer J1.5 (Pin_5)
- net PGED1: now also J1.5 (Pin_5); no longer J1.4 (Pin_4)
- net SCK: now also U6.37 (RC4); no longer U6.9 (RB11)
- net at J6.1 (Pin_1): now also U7.8 (SIGOUT); no longer U7.7 (SIGIN)
- net at J6.2 (Pin_2): now also U7.7 (SIGIN); no longer U7.8 (SIGOUT)
- net +5V renamed V_OUT_DCDC
- net RB15 renamed LED
- net LED: now also U6.44 (RB8); no longer U6.41 (RB5)
- no-connect marks 29 -> 28

Commit message: Avenç de placement
Connections:
- net INA: now also U6.32 (RA8); no longer U6.13 (RA7)
- net INB: now also U6.33 (RB4); no longer U6.32 (RA8)
- net PWM: now also U6.34 (RA4); no longer U6.33 (RB4)
Changed lines of the file:
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@@
-	)
-	(no_connect
-		(at 180.34 81.28)
 	)
 	(no_connect
@@
 	(no_connect
 		(at 52.07 161.29)
+	)
+	(no_connect
+		(at 182.88 86.36)
 	)
 	(no_connect
@@
 	(global_label "PWM"
 		(shape output)
-		(at 130.81 81.28 180)
-		(fields_autoplaced yes)
-		(effects
-			(font
-				(size 1.27 1.27)
-			)
-			(justify right)
-		)
-		(property "Intersheetrefs" "${INTERSHEET_REFS}"
-			(at 123.652 81.28 0)
-			(effects
-				(font
-					(size 1.27 1.27)
-				)
-				(justify right)
+		(at 180.34 81.28 0)
+		(fields_autoplaced yes)
+		(effects
+			(font
+				(size 1.27 1.27)
+			)
+			(justify left)
+		)
+		(property "Intersheetrefs" "${INTERSHEET_REFS}"
+			(at 187.498 81.28 0)
+			(effects
+				(font
+					(size 1.27 1.27)
+				)
+				(justify left)
 				(hide yes)
 			)
@@
 		)
 	)
-	(global_label "INB"
-		(shape output)
-		(at 182.88 88.9 0)
-		(fields_autoplaced yes)
-		(effects
-			(font
-				(size 1.27 1.27)
-			)
-			(justify left)
-		)
-		(property "Intersheetrefs" "${INTERSHEET_REFS}"
-			(at 189.0705 88.9 0)
-			(effects
-				(font
-					(size 1.27 1.27)
-				)
-				(justify left)
-				(hide yes)
-			)
-		)
-	)
 	(global_label "IRQ"
 		(shape input)
@@
 		)
 	)
+	(global_label "INB"
+		(shape output)
+		(at 130.81 81.28 180)
+		(fields_autoplaced yes)
+		(effects
+			(font
+				(size 1.27 1.27)
+			)
+			(justify right)
+		)
+		(property "Intersheetrefs" "${INTERSHEET_REFS}"
+			(at 124.6195 81.28 0)
+			(effects
+				(font
+					(size 1.27 1.27)
+				)
+				(justify right)
+				(hide yes)
+			)
+		)
+	)
 	(global_label "OPEN_FC"
 		(shape input)
@@
 	(global_label "INA"
 		(shape output)
-		(at 182.88 86.36 0)
+		(at 182.88 88.9 0)
 		(fields_autoplaced yes)
 		(effects
@@
 		)
 		(property "Intersheetrefs" "${INTERSHEET_REFS}"
-			(at 188.8891 86.36 0)
-			(effects
-				(font
+			(at 188.8891 88.9 0)
+			(effects
+				(font

Commit message: alfred guapo
Parts:
- J3, J4: footprint Connector_Dsub:DSUB-9_Pins_Horizontal_P2.77x2.84mm_EdgePinOffset4.94mm_Housed_MountingHolesOffset4.94mm -> Connector_Dsub:DSUB-9_Pins_Horizontal_P2.77x2.54mm_EdgePinOffset9.40mm
Connections:
- net INA: now also U6.33 (RB4); no longer U6.32 (RA8)
- net INB: now also U6.32 (RA8); no longer U6.33 (RB4)
- net OSC1: now also C16.1, U6.30 (OSC1), Y2.2; no longer C14.1, U6.31 (OSC2), Y2.1
- net OSC2: now also C14.1, U6.31 (OSC2), Y2.1; no longer C16.1, U6.30 (OSC1), Y2.2
- no-connect marks 28 -> 29
Changed lines of the file:
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@@
 	)
 	(no_connect
+		(at 180.34 99.06)
+	)
+	(no_connect
 		(at 138.43 78.74)
 	)
@@
 		)
 	)
+	(global_label "INA"
+		(shape output)
+		(at 130.81 81.28 180)
+		(fields_autoplaced yes)
+		(effects
+			(font
+				(size 1.27 1.27)
+			)
+			(justify right)
+		)
+		(property "Intersheetrefs" "${INTERSHEET_REFS}"
+			(at 124.8009 81.28 0)
+			(effects
+				(font
+					(size 1.27 1.27)
+				)
+				(justify right)
+				(hide yes)
+			)
+		)
+	)
 	(global_label "LED"
 		(shape input)
@@
 		)
 	)
-	(global_label "OSC2"
-		(shape input)
-		(at 189.23 76.2 0)
-		(fields_autoplaced yes)
-		(effects
-			(font
-				(size 1.27 1.27)
-			)
-			(justify left)
-		)
-		(property "Intersheetrefs" "${INTERSHEET_REFS}"
-			(at 197.2347 76.2 0)
-			(effects
-				(font
-					(size 1.27 1.27)
-				)
-				(justify left)
-				(hide yes)
-			)
-		)
-	)
 	(global_label "UART_RX"
 		(shape input)
@@
 		)
 	)
-	(global_label "CAN_RX"
+	(global_label "INB"
 		(shape output)
-		(at 257.81 36.83 90)
+		(at 182.88 88.9 0)
 		(fields_autoplaced yes)
 		(effects
@@
 		)
 		(property "Intersheetrefs" "${INTERSHEET_REFS}"
-			(at 257.81 26.7086 90)
+			(at 189.0705 88.9 0)
 			(effects
 				(font
@@
 		)
 	)
-	(global_label "LED"
-		(shape input)
-		(at 24.13 34.29 90)
+	(global_label "CAN_RX"
+		(shape output)
+		(at 257.81 36.83 90)
 		(fields_autoplaced yes)
 		(effects
@@
 		)
 		(property "Intersheetrefs" "${INTERSHEET_REFS}"
-			(at 24.13 27.8577 90)
+			(at 257.81 26.7086 90)
 			(effects
 				(font
@@
 		)
 	)
-	(global_label "VCC"
+	(global_label "LED"
 		(shape input)
-		(at 73.66 121.92 90)
+		(at 24.13 34.29 90)
 		(fields_autoplaced yes)
 		(effects
@@
 		)
 		(property "Intersheetrefs" "${INTERSHEET_REFS}"
-			(at 73.66 115.3062 90)
+			(at 24.13 27.8577 90)
 			(effects
 				(font
@@
 		)
 	)
-	(global_label "OSC1"
+	(global_label "VCC"
 		(shape input)
-		(at 203.2 78.74 0)
+		(at 73.66 121.92 90)
 		(fields_autoplaced yes)
 		(effects
@@
 		)
 		(property "Intersheetrefs" "${INTERSHEET_REFS}"
-			(at 211.2047 78.74 0)
+			(at 73.66 115.3062 90)
 			(effects
 				(font
@@
 		)
 	)
-	(global_label "INB"
-		(shape output)
-		(at 130.81 81.28 180)
+	(global_label "OPEN_FC"
+		(shape input)
+		(at 181.61 121.92 0)
 		(fields_autoplaced yes)
 		(effects
@@
 				(size 1.27 1.27)
 			)
-			(justify right)
+			(justify left)
 		)
 		(property "Intersheetrefs" "${INTERSHEET_REFS}"
-			(at 124.6195 81.28 0)
+			(at 193.0014 121.92 0)
 			(effects
 				(font
 					(size 1.27 1.27)
 				)
-				(justify right)
+				(justify left)
 				(hide yes)
 			)
 		)
 	)
-	(global_label "OPEN_FC"
+	(global_label "OSC2"
 		(shape input)
-		(at 181.61 121.92 0)
+		(at 203.2 78.74 0)
 		(fields_autoplaced yes)
 		(effects
@@
 		)
 		(property "Intersheetrefs" "${INTERSHEET_REFS}"
-			(at 193.0014 121.92 0)
+			(at 211.2047 78.74 0)
 			(effects
 				(font
@@
 		)
 	)
-	(global_label "INA"
-		(shape output)
-		(at 182.88 88.9 0)
+	(global_label "OSC1"
+		(shape input)
+		(at 189.23 76.2 0)
 		(fields_autoplaced yes)
 		(effects
@@
 		)
 		(property "Intersheetrefs" "${INTERSHEET_REFS}"
-			(at 188.8891 88.9 0)
+			(at 197.2347 76.2 0)
 			(effects
 				(font
@@
 			)
 		)
-		(property "Footprint" "Connector_Dsub:DSUB-9_Pins_Horizontal_P2.77x2.84mm_EdgePinOffset4.94mm_Housed_MountingHolesOffset4.94mm"
+		(property "Footprint" "Connector_Dsub:DSUB-9_Pins_Horizontal_P2.77x2.54mm_EdgePinOffset9.40mm"
 			(at 93.98 76.2 0)
 			(effects
@@
 			)
 		)
-		(property "Footprint" "Connector_Dsub:DSUB-9_Pins_Horizontal_P2.77x2.84mm_EdgePinOffset4.94mm_Housed_MountingHolesOffset4.94mm"
+		(property "Footprint" "Connector_Dsub:DSUB-9_Pins_Horizontal_P2.77x2.54mm_EdgePinOffset9.40mm"
 			(at 250.19 111.76 0)
 			(effects

Commit message: buenas noches alfred
Connections:
- net CLOSED_FC: now also U6.13 (RA7); no longer U6.4 (RC8)
- net DOWN_W: now also U6.11 (RB13); no longer U6.2 (RC6)
- net OPEN_FC: now also U6.12 (RA10); no longer U6.5 (RC9)
- net UART_RX: now also U6.24 (RB3); no longer U6.10 (RB12)
- net UART_TX: now also U6.23 (RB2); no longer U6.11 (RB13)
- net UP_W: now also U6.10 (RB12); no longer U6.3 (RC7)

Commit message: Placement més o menys colocat, i avenç de algunes connexions
Connections:
- net PGEC1: now also U6.27 (RC2); no longer U6.26 (RC1)
- net PGED1: now also U6.26 (RC1); no longer U6.27 (RC2)

Commit message: el RFID me jodio la vida
Parts:
- removed C20: 100n, Capacitor_SMD:C_1206_3216Metric, symbol Device:C
- removed U9: TJA1051TK-3, Package_SON:HVSON-8-1EP_3x3mm_P0.65mm_EP1.6x2.4mm, symbol Interface_CAN_LIN:TJA1051TK-3
- added R14: 10k, Resistor_SMD:R_1206_3216Metric, symbol Device:R
- added U5: SN65HVD230, Package_SO:SOIC-8_3.9x4.9mm_P1.27mm, symbol Interface_CAN_LIN:SN65HVD230
Connections:
- net V_OUT_DCDC is gone; now on net VCC: C21.1
- net CAN_RX: now also U5.4 (R)
- net CAN_TX: now also U5.1 (D)
- net GND: now also R14.2, U5.2 (GND)
- net PGEC1: now also J1.5 (Pin_5), U6.24 (RB3); no longer J1.4 (Pin_4), U6.27 (RC2)
- net PGED1: now also J1.4 (Pin_4), U6.23 (RB2); no longer J1.5 (Pin_5), U6.26 (RC1)
- net UART_RX: now also U6.26 (RC1); no longer U6.24 (RB3)
- net UART_TX: now also U6.27 (RC2); no longer U6.23 (RB2)
- net VCC: now also U5.3 (VCC)
- net at J4.2, R11.2: now also U5.6 (CANL)
- net at J4.7, R11.1: now also U5.7 (CANH)
- new net: R14.1, U5.8 (Rs)
- no-connect marks 29 -> 31

Commit message: fet
Connections:
- net MISO: now also U6.34 (RA4); no longer U6.43 (RB7)
- net PWM: now also U6.43 (RB7); no longer U6.34 (RA4)
- net at J6.3 (Pin_3): now also U7.20 (AUX2); no longer U7.19 (AUX1)
- net at J6.4 (Pin_4): now also U7.19 (AUX1); no longer U7.20 (AUX2)
Changed lines of the file:
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@@
+	(wire
+		(pts
+			(xy 109.22 160.02) (xy 121.92 160.02)
+		)
+		(stroke
+			(width 0)
+			(type default)
+		)
+	)
 	(wire
 		(pts
@@
 	(wire
 		(pts
+			(xy 111.76 157.48) (xy 121.92 157.48)
+		)
+		(stroke
+			(width 0)
+			(type default)
+		)
+	)
+	(wire
+		(pts
 			(xy 133.35 83.82) (xy 138.43 83.82)
 		)
@@
 	(wire
 		(pts
+			(xy 107.95 157.48) (xy 109.22 157.48)
+		)
+		(stroke
+			(width 0)
+			(type default)
+		)
+	)
+	(wire
+		(pts
 			(xy 259.08 38.1) (xy 259.08 45.72)
 		)
@@
 	(wire
 		(pts
+			(xy 109.22 157.48) (xy 109.22 160.02)
+		)
+		(stroke
+			(width 0)
+			(type default)
+		)
+	)
+	(wire
+		(pts
 			(xy 148.59 40.64) (xy 147.32 40.64)
 		)
@@
 	(wire
 		(pts
-			(xy 111.76 166.37) (xy 111.76 160.02)
+			(xy 111.76 157.48) (xy 111.76 166.37)
 		)
 		(stroke
@@
 	(wire
 		(pts
-			(xy 111.76 160.02) (xy 121.92 160.02)
-		)
-		(stroke
-			(width 0)
-			(type default)
-		)
-	)
-	(wire
-		(pts
 			(xy 147.32 40.64) (xy 147.32 35.56)
 		)
@@
 		(pts
 			(xy 267.97 96.52) (xy 267.97 129.54)
-		)
-		(stroke
-			(width 0)
-			(type default)
-		)
-	)
-	(wire
-		(pts
-			(xy 107.95 157.48) (xy 121.92 157.48)
 		)
 		(stroke
@@
 		)
 	)
+	(global_label "MISO"
+		(shape input)
+		(at 180.34 81.28 0)
+		(fields_autoplaced yes)
+		(effects
+			(font
+				(size 1.27 1.27)
+			)
+			(justify left)
+		)
+		(property "Intersheetrefs" "${INTERSHEET_REFS}"
+			(at 187.9214 81.28 0)
+			(effects
+				(font
+					(size 1.27 1.27)
+				)
+				(justify left)
+				(hide yes)
+			)
+		)
+	)
 	(global_label "LED"
 		(shape input)
@@
 		)
 	)
+	(global_label "PWM"
+		(shape output)
+		(at 133.35 88.9 180)
+		(fields_autoplaced yes)
+		(effects
+			(font
+				(size 1.27 1.27)
+			)
+			(justify right)
+		)
+		(property "Intersheetrefs" "${INTERSHEET_REFS}"
+			(at 126.192 88.9 0)
+			(effects
+				(font
+					(size 1.27 1.27)
+				)
+				(justify right)
+				(hide yes)
+			)
+		)
+	)
 	(global_label "MOSI"
 		(shape input)
@@
 		)
 	)
-	(global_label "PWM"
-		(shape output)
-		(at 180.34 81.28 0)
-		(fields_autoplaced yes)
-		(effects
-			(font
-				(size 1.27 1.27)
-			)
-			(justify left)
-		)
-		(property "Intersheetrefs" "${INTERSHEET_REFS}"
-			(at 187.498 81.28 0)
-			(effects
-				(font
-					(size 1.27 1.27)
-				)
-				(justify left)
-				(hide yes)
-			)
-		)
-	)
 	(global_label "INB"
 		(shape output)
@@
 			(effects
 				(font
-					(size 1.27 1.27)
-				)
-				(justify right)
-				(hide yes)
-			)
-		)
-	)
-	(global_label "MISO"
-		(shape input)
-		(at 133.35 88.9 180)
-		(fields_autoplaced yes)
-		(effects
-			(font
-				(size 1.27 1.27)
-			)
-			(justify right)
-		)
-		(property "Intersheetrefs" "${INTERSHEET_REFS}"
-			(at 125.7686 88.9 0)
-			(effects
-				(font
