File: KiCad/requena.abanto_projecte_vidres/requena.abanto_projecte_vidres.kicad_pcb (KiCad board)
At the start: 4 copper layers, 79 parts, among them J1 Conn_01x05, J3 DE9_Pins, J4 DE9_Pins, J5 Conn_01x02, J6 Conn_01x04, P1 282837-2, P2 282837-2, SW1 SW_Push_SPDT, SW2 SW_Push, SW3 SW_Omron_B3FS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

Commit message: pierreiedgarilofu
Parts:
- moved D5 99.2 mm to (161.6, 46.8), turned to 180 degrees
- moved D9 84.1 mm to (146.5, 52.6)
- moved P1 28.5 mm to (179.6, 30.8)
- moved P2 19.0 mm to (149.0, 30.3)
Changed lines of the file:
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@@
 	(footprint "Diode_THT:D_DO-201AD_P15.24mm_Horizontal"
 		(layer "F.Cu")
-		(at 155.91 -52.29)
+		(at 161.645 46.775 180)
 		(descr "Diode, DO-201AD series, Axial, Horizontal, pin pitch=15.24mm, length*diameter=9.5*5.2mm^2, http://www.diodes.com/_files/packages/DO-201AD.pdf")
 		(tags "Diode DO-201AD series Axial Horizontal pin pitch 15.24mm  length 9.5mm diameter 5.2mm")
@@
 		)
 		(property "Sim.Device" "D"
-			(at 0 0 0)
+			(at 0 0 180)
 			(unlocked yes)
 			(layer "F.Fab")
@@
 		)
 		(property "Sim.Pins" "1=K 2=A"
-			(at 0 0 0)
+			(at 0 0 180)
 			(unlocked yes)
 			(layer "F.Fab")
@@
 		(attr through_hole)
 		(fp_line
-			(start 1.84 0)
-			(end 2.75 0)
+			(start 13.4 0)
+			(end 12.49 0)
 			(stroke
 				(width 0.12)
@@
 		)
 		(fp_line
-			(start 4.175 -2.72)
-			(end 4.175 2.72)
+			(start 4.415 -2.72)
+			(end 4.415 2.72)
 			(stroke
 				(width 0.12)
@@
 		)
 		(fp_line
-			(start 4.415 -2.72)
-			(end 4.415 2.72)
+			(start 4.175 -2.72)
+			(end 4.175 2.72)
 			(stroke
 				(width 0.12)
@@
 		)
 		(fp_line
-			(start 13.4 0)
-			(end 12.49 0)
+			(start 1.84 0)
+			(end 2.75 0)
 			(stroke
 				(width 0.12)
@@
 		)
 		(fp_line
-			(start 0 0)
-			(end 2.87 0)
+			(start 15.24 0)
+			(end 12.37 0)
 			(stroke
 				(width 0.1)
@@
 		)
 		(fp_line
-			(start 4.195 -2.6)
-			(end 4.195 2.6)
+			(start 4.395 -2.6)
+			(end 4.395 2.6)
 			(stroke
 				(width 0.1)
@@
 		)
 		(fp_line
-			(start 4.395 -2.6)
-			(end 4.395 2.6)
+			(start 4.195 -2.6)
+			(end 4.195 2.6)
 			(stroke
 				(width 0.1)
@@
 		)
 		(fp_line
-			(start 15.24 0)
-			(end 12.37 0)
+			(start 0 0)
+			(end 2.87 0)
 			(stroke
 				(width 0.1)
@@
 		)
 		(pad "1" thru_hole roundrect
-			(at 0 0)
+			(at 0 0 180)
 			(size 3.2 3.2)
 			(drill 1.6)
@@
 		)
 		(pad "2" thru_hole circle
-			(at 15.24 0)
+			(at 15.24 0 180)
 			(size 3.2 3.2)
 			(drill 1.6)
@@
 	(footprint "282837-2:TE_282837-2"
 		(layer "F.Cu")
-		(at 151.08 31.15)
+		(at 179.585 30.775)
 		(property "Reference" "P1"
 			(at -1.127255 -5.614945 0)
@@
 	(footprint "Diode_THT:D_DO-201AD_P15.24mm_Horizontal"
 		(layer "F.Cu")
-		(at 155.75 -30.92)
+		(at 146.535 52.65)
 		(descr "Diode, DO-201AD series, Axial, Horizontal, pin pitch=15.24mm, length*diameter=9.5*5.2mm^2, http://www.diodes.com/_files/packages/DO-201AD.pdf")
 		(tags "Diode DO-201AD series Axial Horizontal pin pitch 15.24mm  length 9.5mm diameter 5.2mm")
@@
 	(footprint "282837-2:TE_282837-2"
 		(layer "F.Cu")
-		(at 167.98 31.08)
+		(at 148.985 30.3)
 		(property "Reference" "P2"
 			(at -1.127255 -5.614945 0)
@@
 		(min_thickness 0.25)
 		(filled_areas_thickness no)
-		(fill
+		(fill yes
 			(thermal_gap 0.5)
 			(thermal_bridge_width 0.5)
@@
 		(min_thickness 0.25)
 		(filled_areas_thickness no)
-		(fill
+		(fill yes
 			(thermal_gap 0.5)
 			(thermal_bridge_width 0.5)
@@
 		(min_thickness 0.25)
 		(filled_areas_thickness no)
-		(fill
+		(fill yes
 			(thermal_gap 0.5)
 			(thermal_bridge_width 0.5)
@@
 		(min_thickness 0.25)
 		(filled_areas_thickness no)
-		(fill
+		(fill yes
 			(thermal_gap 0.5)
 			(thermal_bridge_width 0.5)
@@
 	)
 	(zone
+		(net 82)
+		(net_name "OUTM1")
+		(layer "F.Cu")
+		(hatch edge 0.5)
+		(priority 1)
+		(connect_pads
+			(clearance 0.5)
+		)
+		(min_thickness 0.25)
+		(filled_areas_thickness no)
+		(fill yes
+			(thermal_gap 0.5)
+			(thermal_bridge_width 0.5)
+		)
+		(polygon
+			(pts
+				(xy 129.6 51.85) (xy 150.1 51.75) (xy 150.075 53.525) (xy 129.55 53.625)
+			)
+		)
+	)
+	(zone
 		(net 2)
 		(net_name "GNDPWR")
@@
 		(min_thickness 0.25)
 		(filled_areas_thickness no)
-		(fill
+		(fill yes
 			(thermal_gap 0.5)
 			(thermal_bridge_width 0.5)
@@
 		(min_thickness 0.25)
 		(filled_areas_thickness no)
-		(fill
+		(fill yes
 			(thermal_gap 0.5)
 			(thermal_bridge_width 0.5)
@@
 		(min_thickness 0.25)
 		(filled_areas_thickness no)
-		(fill
+		(fill yes
 			(thermal_gap 0.5)
 			(thermal_bridge_width 0.5)
@@
 	)
 	(zone
+		(net 82)
+		(net_name "OUTM1")
+		(layer "F.Cu")
+		(hatch edge 0.5)
+		(priority 1)
+		(connect_pads
+			(clearance 0.5)
+		)
+		(min_thickness 0.25)
+		(filled_areas_thickness no)
+		(fill yes
+			(thermal_gap 0.5)
+			(thermal_bridge_width 0.5)
+		)
+		(polygon
+			(pts
+				(xy 145.740907 54.610955) (xy 145.540907 29.210955) (xy 147.165907 29.185955) (xy 147.365907 54.610955)
+			)
+		)
+	)
+	(zone
 		(net 11)
 		(net_name "V_BAT")
@@
 		(min_thickness 0.25)
 		(filled_areas_thickness no)
-		(fill
+		(fill yes
 			(thermal_gap 0.5)
 			(thermal_bridge_width 0.5)
@@
 		(min_thickness 0.25)
 		(filled_areas_thickness no)
-		(fill
+		(fill yes
 			(thermal_gap 0.5)
 			(thermal_bridge_width 0.5)
@@
 		(min_thickness 0.25)
 		(filled_areas_thickness no)
-		(fill
+		(fill yes
 			(thermal_gap 0.5)
 			(thermal_bridge_width 0.5)
@@
 		(min_thickness 0.25)
 		(filled_areas_thickness no)
-		(fill
+		(fill yes
 			(thermal_gap 0.5)
 			(thermal_bridge_width 0.5)
@@
 		(min_thickness 0.25)
 		(filled_areas_thickness no)
-		(fill
+		(fill yes
 			(thermal_gap 0.5)
 			(thermal_bridge_width 0.5)
@@
 		(min_thickness 0.25)
 		(filled_areas_thickness no)
-		(fill
+		(fill yes
 			(thermal_gap 0.5)
 			(thermal_bridge_width 0.5)

Commit message: buenas noches alfred
Parts:
- moved J3 323.7 mm to (251.7, 159.2), turned to 90 degrees
- moved C12 267.2 mm to (253.2, 126.1)
- moved C18 267.2 mm to (253.2, 129.5)
- moved C19 267.2 mm to (253.2, 132.8)
- moved J1 242.4 mm to (230.9, 136.3), turned to 90 degrees
- moved R6 227.5 mm to (219.2, 101.6), turned to -90 degrees
- moved JP1 227.5 mm to (225.2, 94.8), turned to 90 degrees
- moved R5 225.8 mm to (213.5, 101.9), turned to -90 degrees
- moved SW1 220.6 mm to (206.4, 102.0)
- moved R4 218.5 mm to (199.9, 101.8), turned to -90 degrees
- moved SW2 202.5 mm to (227.2, 102.1)
- moved SW4 199.4 mm to (191.2, 101.9), turned to 180 degrees
- moved R8 197.2 mm to (183.6, 101.3), turned to -90 degrees
- moved C10 195.9 mm to (93.9, 143.1)
- moved C11 195.9 mm to (93.9, 146.4)
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Connections:
- P2 pad 1: OUTM1 -> OUTM2
- P2 pad 2: OUTM2 -> OUTM1
- U6 pad 10: UART_RX -> UP_W
- U6 pad 11: UART_TX -> DOWN_W
- U6 pad 12: unconnected-(U6-RA10-Pad12) -> OPEN_FC
- U6 pad 13: unconnected-(U6-RA7-Pad13) -> CLOSED_FC
- U6 pad 2: DOWN_W -> unconnected-(U6-RC6-Pad2)
- U6 pad 23: unconnected-(U6-RB2-Pad23) -> UART_TX
- U6 pad 24: unconnected-(U6-RB3-Pad24) -> UART_RX
- U6 pad 3: UP_W -> unconnected-(U6-RC7-Pad3)
- U6 pad 4: CLOSED_FC -> unconnected-(U6-RC8-Pad4)
- U6 pad 5: OPEN_FC -> unconnected-(U6-RC9-Pad5)
Routing:
- net OUTM1: track 0.00 -> 82.4 mm
- net OUTM2: track 0.00 -> 62.0 mm
- net Net-(JP1-C): track 0.00 -> 61.5 mm
- net CLOSED_FC: track 0.00 -> 51.2 mm
- net OUTM3: track 0.00 -> 43.3 mm
- net OPEN_D: track 0.00 -> 42.9 mm
- net OPEN_FC: track 0.00 -> 41.8 mm
- net CLOSE_D: track 0.00 -> 36.8 mm
- net DOWN_W: track 0.00 -> 36.6 mm
- net OUTM4: track 0.00 -> 34.7 mm
- net UP_W: track 0.00 -> 32.0 mm
- net GND: track 23.3 -> 55.2 mm, vias 23 -> 42
- net VCC: track 5.12 -> 29.8 mm, vias 19 -> 33
- net Net-(JP1-B): track 0.00 -> 18.3 mm
- net OSC2: track 0.00 -> 11.0 mm
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- removed copper zone on F.Cu, net OUTM1

Commit message: Placement més o menys colocat, i avenç de algunes connexions
Parts:
- removed the C2 at (52.7, 190.4)
- moved J4 219.5 mm to (240.8, 104.1)
- moved J6 190.9 mm to (212.5, 61.5), turned to 90 degrees
- moved U7 184.7 mm to (215.2, 51.2)
- moved Y1 183.5 mm to (215.1, 44.6)
- moved C13 177.4 mm to (219.8, 42.1)
- moved C15 175.9 mm to (211.6, 42.2), turned to 180 degrees
- moved C11 169.4 mm to (226.4, 40.8), turned to 180 degrees
- moved C10 165.3 mm to (226.4, 44.2), turned to 180 degrees
- moved C9 161.4 mm to (226.4, 47.5), turned to 180 degrees
- moved C8 157.7 mm to (226.4, 50.9), turned to 180 degrees
- moved C7 154.1 mm to (226.4, 54.2), turned to 180 degrees
- moved U9 153.0 mm to (214.7, 98.1)
- moved C20 134.1 mm to (214.6, 101.3)
- moved R11 133.1 mm to (219.2, 98.0), turned to -90 degrees
- moved C21 132.0 mm to (209.8, 100.0), turned to 90 degrees
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Connections:
- U6 pad 26: PGEC1 -> PGED1
- U6 pad 27: PGED1 -> PGEC1
Routing:
- net Net-(JP1-C): track 61.5 -> 20.5 mm
- net CLOSED_FC: track 51.2 -> 17.9 mm
- net OPEN_FC: track 41.8 -> 26.8 mm
- net DOWN_W: track 36.6 -> 24.2 mm
- net LED: track 0.00 -> 12.2 mm
- net GND: track 55.2 -> 61.0 mm, vias 42 -> 45
- net OPEN_D: track 42.9 -> 37.3 mm
- net VCC: track 29.8 -> 32.9 mm, vias 33 -> 35
- net Net-(D4-A): track 0.00 -> 2.65 mm
- net CLOSE_D: track 36.8 -> 39.3 mm
- net Net-(D3-A): track 0.00 -> 2.50 mm
- net UP_W: track 32.0 -> 29.6 mm
- net Net-(JP1-B): track 18.3 -> 16.9 mm
- net PGED1: track 0.00 -> 0.74 mm
- net PGEC1: track 0.00 -> 0.74 mm

Commit message: el RFID me jodio la vida
Parts:
- removed C20: 100n, Capacitor_SMD:C_1206_3216Metric
- removed U9: TJA1051TK-3, Package_SON:HVSON-8-1EP_3x3mm_P0.65mm_EP1.6x2.4mm
- added R14: 10k, Resistor_SMD:R_1206_3216Metric, F.Cu at (214.9, 90.7)
- added U5: SN65HVD230, Package_SO:SOIC-8_3.9x4.9mm_P1.27mm, F.Cu at (210.4, 95.2)
- moved Y1 46.3 mm to (260.0, 55.8)
- moved C13 46.3 mm to (264.8, 53.2)
- moved C15 46.3 mm to (256.5, 53.3)
- moved C12 46.3 mm to (271.3, 68.9)
- moved C10 46.3 mm to (271.3, 55.3)
- moved C11 46.3 mm to (271.3, 51.9)
- moved C7 46.3 mm to (271.3, 65.3)
- moved C8 46.3 mm to (271.3, 62.0)
- moved C9 46.3 mm to (271.3, 58.6)
- moved J6 32.1 mm to (214.4, 29.5), turned to -90 degrees
- moved C18 23.3 mm to (165.8, 88.6)
- moved R4 20.7 mm to (164.4, 93.8), turned to -90 degrees
- moved C19 19.0 mm to (174.4, 88.4), turned to -90 degrees
- moved R7 16.5 mm to (136.7, 103.4)
- moved SW3 16.5 mm to (145.3, 104.4)
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Connections:
- C21 pad 1: V_OUT_DCDC -> VCC
- J1 pad 4: PGEC1 -> PGED1
- J1 pad 5: PGED1 -> PGEC1
- U6 pad 23: UART_TX -> PGED1
- U6 pad 24: UART_RX -> PGEC1
- U6 pad 26: PGED1 -> UART_RX
- U6 pad 27: PGEC1 -> UART_TX
Routing:
- net UART_TX: track 0.00 -> 66.0 mm
- net UART_RX: track 0.00 -> 64.9 mm
- net CAN_RX: track 0.00 -> 36.9 mm
- net CAN_TX: track 0.00 -> 34.1 mm
- net Net-(J6-Pin_1): track 0.00 -> 23.3 mm
- net Net-(U5-CANH): track 0.00 -> 21.9 mm
- net Net-(U5-CANL): track 0.00 -> 20.6 mm
- net GND: track 61.0 -> 79.2 mm, vias 45 -> 98
- net PGEC1: track 0.74 -> 16.4 mm
- net PGED1: track 0.74 -> 16.0 mm
- net OPEN_FC: track 26.8 -> 13.4 mm
- net VCC: track 32.9 -> 45.7 mm, vias 35 -> 43
- net UP_W: track 29.6 -> 42.2 mm
- net DOWN_W: track 24.2 -> 35.8 mm
- net Net-(J1-Pin_1): track 0.00 -> 9.76 mm
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Other:
- board outline added: 150.4 x 87.4 mm

Commit message: viva el peru
Routing:
- net AN0: track 1.27 -> 77.0 mm
- net CLOSE_D: track 35.6 -> 34.8 mm
Changed lines of the file:
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@@
-	)
-	(segment
-		(start 167.233156 80.63)
-		(end 168.0275 80.63)
-		(width 0.2)
-		(layer "F.Cu")
-		(net 43)
 	)
 	(segment
@@
 		(layer "F.Cu")
 		(net 44)
+	)
+	(segment
+		(start 175.29 76.328944)
+		(end 172.567056 73.606)
+		(width 0.2)
+		(layer "F.Cu")
+		(net 52)
+	)
+	(segment
+		(start 147.773443 74.3935)
+		(end 124.345943 50.966)
+		(width 0.2)
+		(layer "F.Cu")
+		(net 52)
+	)
+	(segment
+		(start 175.29 83.8925)
+		(end 175.29 76.328944)
+		(width 0.2)
+		(layer "F.Cu")
+		(net 52)
+	)
+	(segment
+		(start 172.567056 73.606)
+		(end 157.534 73.606)
+		(width 0.2)
+		(layer "F.Cu")
+		(net 52)
 	)
 	(segment
@@
 	)
 	(segment
+		(start 157.534 73.606)
+		(end 156.7465 74.3935)
+		(width 0.2)
+		(layer "F.Cu")
+		(net 52)
+	)
+	(segment
+		(start 156.7465 74.3935)
+		(end 147.773443 74.3935)
+		(width 0.2)
+		(layer "F.Cu")
+		(net 52)
+	)
+	(segment
+		(start 119.1085 50.966)
+		(end 118.535 50.3925)
+		(width 0.2)
+		(layer "F.Cu")
+		(net 52)
+	)
+	(segment
+		(start 124.345943 50.966)
+		(end 119.1085 50.966)
+		(width 0.2)
+		(layer "F.Cu")
+		(net 52)
+	)
+	(segment
 		(start 207.89 97.06)
 		(end 198.002 97.06)
@@
 		(min_thickness 0.25)
 		(filled_areas_thickness no)
-		(fill
+		(fill yes
 			(thermal_gap 0.5)
 			(thermal_bridge_width 0.5)
@@
 		(min_thickness 0.25)
 		(filled_areas_thickness no)
-		(fill
+		(fill yes
 			(thermal_gap 0.5)
 			(thermal_bridge_width 0.5)
@@
 		(min_thickness 0.25)
 		(filled_areas_thickness no)
-		(fill
+		(fill yes
 			(thermal_gap 0.5)
 			(thermal_bridge_width 0.5)
@@
 		(min_thickness 0.25)
 		(filled_areas_thickness no)
-		(fill
+		(fill yes
 			(thermal_gap 0.5)
 			(thermal_bridge_width 0.5)
@@
 		(min_thickness 0.25)
 		(filled_areas_thickness no)
-		(fill
+		(fill yes
 			(thermal_gap 0.5)
 			(thermal_bridge_width 0.5)
@@
 		(min_thickness 0.25)
 		(filled_areas_thickness no)
-		(fill
+		(fill yes
 			(thermal_gap 0.5)
 			(thermal_bridge_width 0.5)
@@
 		(min_thickness 0.25)
 		(filled_areas_thickness no)
-		(fill
+		(fill yes
 			(thermal_gap 0.5)
 			(thermal_bridge_width 0.5)
@@
 		(min_thickness 0.25)
 		(filled_areas_thickness no)
-		(fill
+		(fill yes
 			(thermal_gap 0.5)
 			(thermal_bridge_width 0.5)
@@
 		(min_thickness 0.25)
 		(filled_areas_thickness no)
-		(fill
+		(fill yes
 			(thermal_gap 0.5)
 			(thermal_bridge_width 0.5)
@@
 		(min_thickness 0.25)
 		(filled_areas_thickness no)
-		(fill
+		(fill yes
 			(thermal_gap 0.5)
 			(thermal_bridge_width 0.5)
@@
 		(min_thickness 0.25)
 		(filled_areas_thickness no)
-		(fill
+		(fill yes
 			(thermal_gap 0.5)
 			(thermal_bridge_width 0.5)
@@
 		(min_thickness 0.25)
 		(filled_areas_thickness no)
-		(fill
-			(thermal_gap 0.5)
-			(thermal_bridge_width 0.5)
+		(fill yes
+			(thermal_gap 0.5)
+			(thermal_bridge_width 0.5)

Commit message: .
Parts:
- moved R3 5.11 mm to (109.8, 46.5), turned to 180 degrees
- moved R2 4.32 mm to (108.1, 51.0), turned to -90 degrees
- moved C14 4.23 mm to (185.7, 74.7), turned to 0 degrees
- moved C16 4.13 mm to (185.7, 78.2), turned to 0 degrees
- moved Y2 3.82 mm to (182.4, 76.5)
Routing:
- net AN0: track 77.0 -> 1.27 mm
- net AMPLIFICADO: track 0.00 -> 28.4 mm
- net Net-(U3A--): track 8.84 -> 14.6 mm
- net OSC2: track 11.0 -> 5.92 mm
- net OSC1: track 10.9 -> 6.09 mm
- net UART_TX: track 66.0 -> 62.5 mm
- net UART_RX: track 64.9 -> 62.3 mm
- net GND: track 79.2 -> 80.7 mm, vias 98 -> 69
- net VCC: track 45.7 -> 47.2 mm, vias 43 -> 44
- removed copper zone on F.Cu, net AMPLIFICADO

Commit message: millora
Parts:
- moved C13 46.9 mm to (217.9, 54.7), turned to -90 degrees
- moved Y1 44.7 mm to (215.5, 52.5), turned to -90 degrees
- moved C15 38.7 mm to (218.0, 50.2), turned to 90 degrees
- moved J6 6.96 mm to (207.7, 27.6), turned to 90 degrees
- moved U7 1.15 mm to (210.2, 52.6), turned to 0 degrees
Routing:
- net Net-(J6-Pin_2): track 0.00 -> 29.0 mm
- net Net-(J6-Pin_1): track 23.3 -> 29.3 mm
- net Net-(U7-OSCIN): track 0.00 -> 5.88 mm
- net Net-(U7-OSCOUT): track 0.00 -> 5.62 mm
- net NRSTPD: track 0.00 -> 0.56 mm

Commit message: -
Parts:
- moved C12 61.2 mm to (212.8, 50.7), turned to 90 degrees
- moved C13 9.08 mm to (219.7, 45.8), turned to 0 degrees
- moved Y1 7.99 mm to (216.4, 44.6)
- moved U7 7.68 mm to (210.9, 45.0)
- moved C15 7.18 mm to (219.7, 43.3), turned to 0 degrees
Routing:
- net Net-(J6-Pin_1): track 29.3 -> 22.9 mm
- net Net-(J6-Pin_2): track 29.0 -> 22.8 mm
- net GND: track 80.7 -> 85.9 mm, vias 69 -> 74
- net VCC: track 47.2 -> 49.4 mm, vias 44 -> 46
- net Net-(U7-VMID): track 0.00 -> 1.90 mm
- net NRSTPD: track 0.56 -> 1.68 mm, vias 0 -> 1
