File: KiCad/requena.abanto_projecte_vidres/requena.abanto_projecte_vidres.kicad_pcb (KiCad board)
At the start: 4 copper layers, 150.4 x 87.4 mm, 78 parts, among them J1 Conn_01x05, J3 DE9_Pins, J4 DE9_Pins, J5 Conn_01x02, J6 Conn_01x04, P1 282837-2, P2 282837-2, SW1 SW_Push_SPDT, SW2 SW_Push, SW3 SW_Omron_B3FS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

Commit message: fet
Parts:
- moved C11 64.1 mm to (207.2, 50.6), turned to 90 degrees
- moved C10 62.8 mm to (210.9, 38.1), turned to -90 degrees
- moved C9 59.3 mm to (215.6, 38.2), turned to -90 degrees
- moved C7 57.9 mm to (220.1, 38.2), turned to -90 degrees
- moved C8 53.9 mm to (218.4, 51.7), turned to 90 degrees
- moved C12 1.06 mm to (212.9, 51.8)
Connections:
- U6 pad 34: PWM -> MISO
- U6 pad 43: MISO -> PWM
- U7 pad 19: Net-(J6-Pin_3) -> Net-(J6-Pin_4)
- U7 pad 20: Net-(J6-Pin_4) -> Net-(J6-Pin_3)
Routing:
- net AN0: track 1.27 -> 73.8 mm, vias 0 -> 2
- net INB: track 0.00 -> 60.6 mm, vias 0 -> 1
- net PWM: track 0.00 -> 59.3 mm
- net INA: track 0.00 -> 55.4 mm, vias 0 -> 1
- net MISO: track 0.00 -> 52.6 mm
- net IRQ: track 0.00 -> 51.9 mm, vias 0 -> 2
- net SCK: track 0.00 -> 50.0 mm
- net MOSI: track 0.00 -> 49.9 mm
- net NRSTPD: track 1.68 -> 48.6 mm, vias 1 -> 2
- net Net-(J6-Pin_3): track 0.00 -> 41.6 mm
- net Net-(J6-Pin_4): track 0.00 -> 40.9 mm
- net GND: track 85.9 -> 109.0 mm, vias 74 -> 103
- net VCC: track 49.4 -> 70.8 mm, vias 46 -> 60
- net Net-(U7-VMID): track 1.90 -> 2.99 mm

Commit message: hamza zibar
Routing:
- net GND: track 109.0 -> 113.6 mm
Changed lines of the file:
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@@
 	)
 	(segment
+		(start 210.94 44.96)
+		(end 211.69 45.71)
+		(width 0.2)
+		(layer "F.Cu")
+		(net 4)
+	)
+	(segment
 		(start 149.2675 108.16)
 		(end 149.2675 108.2)
@@
 	)
 	(segment
-		(start 207.44 44.71)
-		(end 207.43 44.72)
-		(width 0.2)
-		(layer "F.Cu")
-		(net 4)
-	)
-	(segment
 		(start 141.5775 85.65)
 		(end 141.5775 87.1775)
@@
 	)
 	(segment
+		(start 208.5025 45.21)
+		(end 206.38 45.21)
+		(width 0.2)
+		(layer "F.Cu")
+		(net 4)
+	)
+	(segment
 		(start 207.15 52.045)
 		(end 208.645 52.045)
@@
 	)
 	(segment
+		(start 206.38 45.21)
+		(end 206.35 45.18)
+		(width 0.2)
+		(layer "F.Cu")
+		(net 4)
+	)
+	(segment
 		(start 220.115 53.145)
 		(end 220.12 53.14)
@@
 	)
 	(segment
-		(start 118.11 92.68835)
-		(end 118.11 91.415)
-		(width 0.5)
-		(layer "F.Cu")
-		(net 4)
-	)
-	(segment
-		(start 208.505 43.21)
-		(end 207.47 43.21)
+		(start 211.69 47.3975)
+		(end 211.69 49.13)
 		(width 0.2)
 		(layer "F.Cu")
@@
 	)
 	(segment
-		(start 209.6925 47.3975)
-		(end 209.6925 48.4425)
-		(width 0.2)
+		(start 118.11 92.68835)
+		(end 118.11 91.415)
+		(width 0.5)
 		(layer "F.Cu")
 		(net 4)
@@
 	)
 	(segment
-		(start 211.69 48.4)
-		(end 211.6925 48.3975)
-		(width 0.2)
-		(layer "F.Cu")
-		(net 4)
-	)
-	(segment
 		(start 180.77 77.43)
 		(end 180.78 77.44)
@@
 	)
 	(segment
-		(start 207.47 43.21)
-		(end 207.46 43.2)
-		(width 0.2)
-		(layer "F.Cu")
-		(net 4)
-	)
-	(segment
 		(start 156.1825 67.55)
 		(end 156.1825 68.95)
@@
 	)
 	(segment
+		(start 208.5025 43.21)
+		(end 206.41 43.21)
+		(width 0.2)
+		(layer "F.Cu")
+		(net 4)
+	)
+	(segment
 		(start 168.0275 78.23)
 		(end 166.62 78.23)
@@
 	)
 	(segment
-		(start 208.505 44.71)
-		(end 207.44 44.71)
-		(width 0.2)
-		(layer "F.Cu")
-		(net 4)
-	)
-	(segment
 		(start 174.36 89.845)
 		(end 175.955 89.845)
@@
 	)
 	(segment
-		(start 209.6925 48.4425)
-		(end 209.7 48.45)
-		(width 0.2)
-		(layer "F.Cu")
-		(net 4)
-	)
-	(segment
 		(start 154.1975 72.47)
 		(end 154.1975 73.7925)
@@
 	)
 	(segment
-		(start 211.6925 47.3975)
-		(end 211.6925 48.3975)
-		(width 0.2)
-		(layer "F.Cu")
-		(net 4)
-	)
-	(segment
 		(start 209.025 101.505)
 		(end 209.02 101.51)
@@
 	)
 	(segment
-		(start 208.505 45.21)
-		(end 207.44 45.21)
-		(width 0.2)
-		(layer "F.Cu")
-		(net 4)
-	)
-	(segment
 		(start 141.2675 106.62)
 		(end 141.2675 108.2)
@@
 	)
 	(segment
+		(start 209.69 47.3975)
+		(end 209.69 48.44)
+		(width 0.2)
+		(layer "F.Cu")
+		(net 4)
+	)
+	(segment
 		(start 119.05 99.275)
 		(end 119.05 97.95)
@@
 	)
 	(segment
+		(start 210.94 44.96)
+		(end 209.69 46.21)
+		(width 0.2)
+		(layer "F.Cu")
+		(net 4)
+	)
+	(segment
 		(start 163.325 79.05)
 		(end 163.325 80.4)
@@
 	)
 	(via micro
-		(at 207.43 45.21)
+		(at 206.35 45.18)
 		(size 0.3)
 		(drill 0.1)
@@
 		(size 0.3)
 		(drill 0.1)
-		(layers "F.Cu" "B.Cu")
+		(layers "F.Cu" "In1.Cu")
 		(net 4)
 	)
@@
 		(net 4)
 	)
+	(via micro
+		(at 206.41 43.21)
+		(size 0.3)
+		(drill 0.1)
+		(layers "F.Cu" "In1.Cu")
+		(net 4)
+	)
 	(via
 		(at 184.86 79.56)
@@
 		(net 4)
 	)
+	(via micro
+		(at 211.69 49.13)
+		(size 0.3)
+		(drill 0.1)
+		(layers "F.Cu" "In1.Cu")
+		(net 4)
+	)
 	(via
 		(at 209.04 98.23)
@@
 	)
 	(via micro
-		(at 207.43 44.72)
+		(at 209.69 48.44)
 		(size 0.3)
 		(drill 0.1)
@@
 		(net 4)
 	)
-	(via micro
-		(at 207.46 43.21)
-		(size 0.3)
-		(drill 0.1)
-		(layers "F.Cu" "In1.Cu")
-		(net 4)
-	)
 	(via
 		(at 163.325 80.4)
@@
 		(net 4)
 	)
-	(via micro
-		(at 211.7 48.41)
-		(size 0.3)
-		(drill 0.1)
-		(layers "F.Cu" "In1.Cu")
-		(net 4)
-	)
 	(via
 		(at 166.62 78.23)
@@
 		(net 4)
 	)
-	(via micro
-		(at 209.675977 48.553316)
-		(size 0.3)
-		(drill 0.1)
-		(layers "F.Cu" "In1.Cu")
-		(net 4)
-	)
 	(via
 		(at 149.4175 97.29)
@@
 	)
 	(via
+		(at 211.85 44.97)
+		(size 0.6)
+		(drill 0.3)
+		(layers "F.Cu" "B.Cu")
+		(net 4)
+	)
+	(via
 		(at 216.3725 92.3525)
 		(size 0.6)
@@
 	)
 	(segment
-		(start 204.88 80.93)
-		(end 204.88 80.91467)
+		(start 206.067335 79.742665)
+		(end 204.88 80.93)
 		(width 0.2)
 		(layer "F.Cu")
@@
 	)
 	(segment
-		(start 179.3525 79.83)
-		(end 179.4425 79.92)
+		(start 206.067335 79.727335)
+		(end 206.067335 79.742665)
 		(width 0.2)
 		(layer "F.Cu")
@@
 	)
 	(segment
-		(start 180.7 79.83)
-		(end 181.8 80.93)
+		(start 179.3525 79.83)
+		(end 179.4425 79.92)
 		(width 0.2)
 		(layer "F.Cu")
@@
 	)
 	(segment
-		(start 204.88 80.91467)
-		(end 206.067335 79.727335)
+		(start 180.7 79.83)
+		(end 181.8 80.93)
 		(width 0.2)
 		(layer "F.Cu")
@@
 	)
 	(segment
-		(start 205.874669 79.92)
-		(end 206.067335 79.727335)
-		(width 0.2)
-		(layer "F.Cu")
-		(net 26)
-	)
-	(segment
 		(start 191.425 102.375)
 		(end 191.33 102.28)
@@
 	)
 	(segment
-		(start 184.92 68.18)
-		(end 184.9 68.18)
-		(width 0.2)
-		(layer "B.Cu")
-		(net 57)
-	)
-	(segment
-		(start 207.39 45.71)
-		(end 184.92 68.18)
-		(width 0.2)
-		(layer "B.Cu")
-		(net 57)
-	)
-	(segment
 		(start 174.07 68.75)
 		(end 173.97 68.85)
@@
 	)
 	(segment
-		(start 184.9 68.18)
-		(end 184.33 68.75)
+		(start 184.35 68.75)
+		(end 174.07 68.75)
 		(width 0.2)
 		(layer "B.Cu")
@@
 	)
 	(segment
-		(start 184.33 68.75)
-		(end 174.07 68.75)
+		(start 207.39 45.71)
+		(end 184.35 68.75)
 		(width 0.2)
 		(layer "B.Cu")
@@
 		(min_thickness 0.25)
 		(filled_areas_thickness no)
-		(fill yes
+		(fill
 			(thermal_gap 0.5)
 			(thermal_bridge_width 0.5)
@@
 		(min_thickness 0.25)
 		(filled_areas_thickness no)
-		(fill yes
+		(fill
 			(thermal_gap 0.5)
 			(thermal_bridge_width 0.5)
@@
 		(min_thickness 0.25)
 		(filled_areas_thickness no)
-		(fill yes
+		(fill
 			(thermal_gap 0.5)
 			(thermal_bridge_width 0.5)
@@
 		(min_thickness 0.25)
 		(filled_areas_thickness no)
-		(fill yes
+		(fill
 			(thermal_gap 0.5)
 			(thermal_bridge_width 0.5)
@@
 		(min_thickness 0.25)
 		(filled_areas_thickness no)
-		(fill yes
+		(fill
 			(thermal_gap 0.5)
 			(thermal_bridge_width 0.5)
@@
 		(min_thickness 0.25)
 		(filled_areas_thickness no)
-		(fill yes
+		(fill
 			(thermal_gap 0.5)
 			(thermal_bridge_width 0.5)
@@
 		(min_thickness 0.25)
 		(filled_areas_thickness no)
-		(fill yes
+		(fill
 			(thermal_gap 0.5)
 			(thermal_bridge_width 0.5)
@@
 		(min_thickness 0.25)
 		(filled_areas_thickness no)
-		(fill yes
+		(fill
 			(thermal_gap 0.5)
 			(thermal_bridge_width 0.5)
@@
 		(min_thickness 0.25)
 		(filled_areas_thickness no)
-		(fill yes
+		(fill
 			(thermal_gap 0.5)
 			(thermal_bridge_width 0.5)
@@
 		(min_thickness 0.25)
 		(filled_areas_thickness no)
-		(fill yes
+		(fill
 			(thermal_gap 0.5)
 			(thermal_bridge_width 0.5)
@@
 		(min_thickness 0.25)
 		(filled_areas_thickness no)
-		(fill yes
+		(fill
 			(thermal_gap 0.5)
 			(thermal_bridge_width 0.5)
@@
 		(min_thickness 0.25)
 		(filled_areas_thickness no)
-		(fill yes
+		(fill
 			(thermal_gap 0.5)
 			(thermal_bridge_width 0.5)

Commit message: regles de disseny i més coses
Parts:
- moved REF** 23.1 mm to (220.7, 108.2)
- moved REF** 23.1 mm to (223.0, 29.3)
- moved J3 18.0 mm to (213.8, 67.4)
- moved J4 17.5 mm to (213.8, 99.7)
- moved R11 12.0 mm to (207.9, 95.1)
- moved U5 9.81 mm to (200.6, 94.5)
- moved C21 9.81 mm to (200.7, 99.2)
- moved R14 9.81 mm to (205.1, 90.0)
- moved R3 7.36 mm to (116.7, 48.9), turned to -90 degrees
- moved U3 6.84 mm to (114.0, 43.2)
- moved C6 4.90 mm to (122.9, 46.4)
- moved R2 4.66 mm to (112.3, 49.0), turned to 90 degrees
- moved C10 3.59 mm to (207.3, 38.1)
- moved C11 3.59 mm to (203.6, 50.5)
- moved C12 3.59 mm to (209.3, 51.8)
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Connections:
- net AMPLIFICADO renamed OUTNOINV
- net Net-(D3-A) renamed LEDPROGRAM
- net Net-(D4-A) renamed LEDVCC
- net Net-(J1-Pin_1) renamed INJUMPER
- net Net-(J6-Pin_1) renamed SIGOUT
- net Net-(J6-Pin_2) renamed SIGIN
- net Net-(J6-Pin_3) renamed AUX2
- net Net-(J6-Pin_4) renamed AUX1
- net Net-(JP1-B) renamed OUTJUMPER
- net Net-(JP1-C) renamed MCLR
- net Net-(U3A-+) renamed OUTSHUNT
- net Net-(U3A--) renamed REALIMENTACION_NOINV
- net Net-(U5-CANH) renamed CAN+
- net Net-(U5-CANL) renamed CAN-
- net Net-(U5-Rs) renamed RSCAN
- net Net-(U6-VCAP) renamed VCAP
- net Net-(U7-OSCIN) renamed OSC2RFID
- net Net-(U7-OSCOUT) renamed OSC1RFID
- net Net-(U7-VMID) renamed VMID
Routing:
- net OUTNOINV: track 28.4 -> 8.93 mm
- net UART_RX: track 62.0 -> 44.2 mm
- net UART_TX: track 62.5 -> 46.0 mm
- net SHUNT: track 14.9 -> 26.8 mm
- net CAN_TX: track 34.1 -> 24.0 mm
- net CAN_RX: track 36.9 -> 27.2 mm
- net OUTSHUNT: track 18.1 -> 9.67 mm
- net CAN-: track 20.6 -> 12.3 mm
- net CAN+: track 21.9 -> 14.1 mm
- net AN0: track 73.8 -> 81.0 mm
- net VCC: track 70.8 -> 65.6 mm
- net SCK: track 50.0 -> 46.4 mm
- net MISO: track 52.6 -> 49.0 mm
- net MOSI: track 49.9 -> 46.3 mm
- net IRQ: track 51.9 -> 48.8 mm
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Other:
- board size 150.4 x 87.4 mm -> 126.4 x 87.4 mm

Commit message: hola alfred
Parts:
- moved C12 63.3 mm to (260.2, 89.4)
- moved C7 63.3 mm to (267.4, 75.7)
- moved C11 63.3 mm to (254.5, 88.1)
- moved C13 63.3 mm to (267.0, 83.3)
- moved C15 63.3 mm to (267.1, 80.8)
- moved C9 63.3 mm to (262.9, 75.7)
- moved U7 63.3 mm to (258.3, 82.5)
- moved C10 63.3 mm to (258.2, 75.7)
- moved C8 63.3 mm to (265.7, 89.2)
- moved Y1 63.3 mm to (263.7, 82.2)
- moved J6 60.9 mm to (252.4, 64.6)
- moved J1 60.7 mm to (229.7, 45.8)
- moved JP1 44.5 mm to (228.5, 104.2)
- moved C19 41.9 mm to (140.4, 63.8), turned to 0 degrees
- moved R6 40.2 mm to (150.7, 132.7)
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Routing:
- net AN0: track 81.0 -> 10.6 mm
- net INB: track 60.6 -> 5.09 mm
- net INA: track 55.4 -> 3.28 mm
- net PWM: track 60.0 -> 10.9 mm
- net MISO: track 49.0 -> 0.13 mm
- net IRQ: track 48.8 -> 0.94 mm, vias 2 -> 1
- net SCK: track 46.4 -> 0.00 mm
- net MOSI: track 46.3 -> 0.06 mm
- net NRSTPD: track 47.4 -> 1.24 mm, vias 2 -> 1
- net UART_TX: track 46.0 -> 0.00 mm
- net UART_RX: track 44.2 -> 0.13 mm
- net DOWN_W: track 35.8 -> 78.1 mm
- net AUX2: track 41.6 -> 1.77 mm
- net AUX1: track 40.9 -> 1.33 mm
- net CAN_RX: track 27.2 -> 0.60 mm
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Other:
- board size 126.4 x 87.4 mm -> 99.5 x 82.4 mm

Commit message: -
Parts:
- removed C10, C11, C12, C7, C8, C9: 100nF, Capacitor_SMD:C_1206_3216Metric
- removed J6: Conn_01x04, Connector_PinHeader_2.54mm:PinHeader_1x04_P2.54mm_Vertical
- removed U7: PN5120A0HN1, Package_DFN_QFN:HVQFN-32-1EP_5x5mm_P0.5mm_EP3.1x3.1mm
- added C20: C_Small, Capacitor_SMD:C_1206_3216Metric, F.Cu at (271.1, 44.7)
- added C26: C_Small, Capacitor_SMD:C_1206_3216Metric, F.Cu at (271.1, 48.0)
- added C27: C_Small, Capacitor_SMD:C_1206_3216Metric, F.Cu at (271.1, 51.4)
- added C28: C_Small, Capacitor_SMD:C_1206_3216Metric, F.Cu at (271.1, 54.8)
- added C29: C_Small, Capacitor_SMD:C_1206_3216Metric, F.Cu at (276.8, 44.7)
- added C30: C_Small, Capacitor_SMD:C_1206_3216Metric, F.Cu at (276.8, 48.0)
- added C31: C_Small, Capacitor_SMD:C_1206_3216Metric, F.Cu at (276.8, 51.4)
- added C32: C_Small, Capacitor_SMD:C_1206_3216Metric, F.Cu at (276.8, 54.8)
- added C34: 100nF, Capacitor_SMD:C_1206_3216Metric, F.Cu at (282.4, 44.7)
- added C35: 100nF, Capacitor_SMD:C_1206_3216Metric, F.Cu at (282.4, 48.0)
- added C36: 100nF, Capacitor_SMD:C_1206_3216Metric, F.Cu at (282.4, 51.4)
- added C37: 100nF, Capacitor_SMD:C_1206_3216Metric, F.Cu at (282.4, 54.8)
- added L1: L, Inductor_SMD:L_1206_3216Metric, F.Cu at (271.2, 58.1)
- added L2: L, Inductor_SMD:L_1206_3216Metric, F.Cu at (271.2, 61.6)
- added L3: L, Inductor_SMD:L_1206_3216Metric, F.Cu at (271.2, 65.0)
- added R15: R, Resistor_SMD:R_1206_3216Metric, F.Cu at (276.9, 58.1)
- added R16: R, Resistor_SMD:R_1206_3216Metric, F.Cu at (276.9, 61.4)
- added R17: R, Resistor_SMD:R_1206_3216Metric, F.Cu at (276.9, 64.7)
- added R18: R, Resistor_SMD:R_1206_3216Metric, F.Cu at (276.9, 68.0)
- moved J1 75.4 mm to (166.9, 87.7)
- moved C13 21.9 mm to (288.9, 83.1)
- moved C15 21.9 mm to (288.9, 80.6)
- moved Y1 21.9 mm to (285.6, 81.9)
Connections:
- U6 pad 42: unconnected-(U6-RB6-Pad42) -> SDA
Routing:
- net GND: track 95.9 -> 60.6 mm, vias 87 -> 71
- net VCC: track 69.6 -> 48.4 mm, vias 63 -> 48
- net VMID: track 2.99 -> 0.00 mm
- net OSC1RFID: track 5.81 -> 3.57 mm
- net OSC2RFID: track 5.94 -> 3.85 mm
- net SIGOUT: track 2.09 -> 0.00 mm
- net SIGIN: track 2.02 -> 0.00 mm
- net AUX2: track 1.77 -> 0.35 mm
- net NRSTPD: track 1.24 -> 0.00 mm, vias 1 -> 0
- net AUX1: track 1.33 -> 0.20 mm
- net IRQ: track 0.94 -> 0.00 mm, vias 1 -> 0
- net PWM: track 10.9 -> 10.1 mm

Commit message: --
Parts:
- added U8: MFRC52201HN1_157, MFRC52201HN1_157:QFN50P500X500X100-33N, F.Cu at (255.2, 52.9)
Routing:
- net (no net): track 0.00 -> 0.55 mm

Commit message: bomboclat walahi
Parts:
- moved C34 117.8 mm to (170.6, 81.7), turned to 90 degrees
- moved C35 114.2 mm to (173.3, 81.7), turned to 90 degrees
- moved C15 112.4 mm to (177.4, 66.9), turned to 90 degrees
- moved C36 110.8 mm to (175.8, 81.7), turned to 90 degrees
- moved C13 110.1 mm to (179.9, 67.0), turned to 90 degrees
- moved Y1 107.5 mm to (178.7, 70.3), turned to 0 degrees
- moved C37 107.4 mm to (178.5, 81.7), turned to 90 degrees
- moved C31 100.1 mm to (183.3, 87.3), turned to 180 degrees
- moved C29 98.8 mm to (187.7, 87.4), turned to -90 degrees
- moved R18 95.0 mm to (182.9, 82.0), turned to -90 degrees
- moved C32 94.9 mm to (182.2, 61.6), turned to 180 degrees
- moved R17 93.1 mm to (183.8, 65.2), turned to -90 degrees
- moved C30 90.2 mm to (187.8, 62.5), turned to 90 degrees
- moved R15 89.0 mm to (191.1, 82.0), turned to 90 degrees
- moved C27 88.9 mm to (187.7, 82.0), turned to -90 degrees
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Connections:
- U8 pad 33: unconnected-(U8-EXP-Pad33) -> GND
Routing:
- net UART_RX: track 0.13 -> 54.3 mm, vias 0 -> 1
- net UART_TX: track 0.00 -> 53.9 mm, vias 0 -> 1
- net SDA: track 0.00 -> 43.1 mm, vias 0 -> 2
- net MOSI: track 0.06 -> 40.3 mm
- net GND: track 60.6 -> 98.7 mm, vias 71 -> 91
- net IRQ: track 0.00 -> 37.5 mm, vias 0 -> 2
- net MISO: track 0.00 -> 35.0 mm
- net Net-(U8-RX): track 0.00 -> 25.5 mm, vias 0 -> 2
- net PGED1: track 0.00 -> 18.5 mm
- net PGEC1: track 0.76 -> 19.2 mm
- net MCLR: track 1.77 -> 17.2 mm
- net Net-(U8-VMID): track 0.00 -> 14.0 mm
- net OUTJUMPER: track 12.3 -> 24.7 mm
- net Net-(C20-Pad1): track 0.00 -> 11.1 mm
- net CAN+: track 4.90 -> 14.6 mm
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
Commit message: v2placement
Parts:
- moved REF** 11.9 mm to (206.4, 33.7)
- moved REF** 8.95 mm to (204.2, 110.1)
- moved REF** 6.13 mm to (105.8, 109.5)
- moved C14 5.61 mm to (156.8, 74.7)
- moved C31 5.61 mm to (185.6, 92.4)
- moved C35 5.61 mm to (175.5, 86.8)
- moved D4 5.61 mm to (135.4, 75.9)
- moved JP1 5.61 mm to (161.5, 86.1)
- moved L3 5.61 mm to (199.0, 80.7)
- moved R11 5.61 mm to (190.3, 98.7)
- moved R12 5.61 mm to (130.4, 72.7)
- moved R15 5.61 mm to (193.4, 87.2)
- moved R16 5.61 mm to (193.3, 74.9)
- moved R17 5.61 mm to (186.1, 70.3)
- moved R7 5.61 mm to (163.2, 105.6)
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Routing:
- net AN0: track 9.30 -> 55.9 mm, vias 1 -> 2
- net NRSTPD: track 0.00 -> 46.4 mm, vias 0 -> 2
- net CAN_RX: track 0.60 -> 40.3 mm, vias 0 -> 2
- net CAN_TX: track 0.00 -> 39.6 mm
- net SCK: track 0.00 -> 38.5 mm, vias 0 -> 2
- net INB: track 5.09 -> 34.0 mm
- net INA: track 3.26 -> 27.8 mm
- net PWM: track 10.1 -> 31.3 mm
- net VCC: track 50.2 -> 50.3 mm, vias 50 -> 55
- net GND: vias 91 -> 94
Other:
- board size 99.5 x 82.4 mm -> 107.8 x 82.4 mm
