File: KiCad/requena.abanto_projecte_vidres/etapa_de_potencia.kicad_sch (KiCad schematic)
At the start: 30 parts, among them J5 Conn_01x02, P1 282837-2, P2 282837-2, U1 L298N, U2 TSR2-2450, U3 MCP6022, U4 LM1117DT-3.3

Commit message: foking diodos
Parts:
- removed C2: 100n, Capacitor_SMD:C_1206_3216Metric, symbol Device:C
- added C2: 470uF, Capacitor_THT:CP_Radial_D4.0mm_P1.50mm, symbol Device:C_Polarized
- added C25: 100n, Capacitor_SMD:C_1206_3216Metric, symbol Device:C
Connections:
- net GND: now also C2.2, C25.2
- net VCC: now also C2.1
- net V_BAT: now also C25.1
- net AMPLIFICADO: now reaches R3.1, U3.1, U3.5 (+)
- net OUTM3: now reaches D11.1 (K), D7.2 (A), U1.13 (OUT3)
- net OUTM3: now also P1.2; no longer P2.1
- net OUTM1: now reaches D5.2 (A), D9.1 (K), U1.2 (OUT1)
- net OUTM1: now also P2.1; no longer P1.1
- net OUTM2: now reaches D10.1 (K), D6.2 (A), U1.3 (OUT2)
- net OUTM2: now also P2.2; no longer P1.2
- net OUTM4: now reaches D12.1 (K), D8.2 (A), U1.14 (OUT4)
- net OUTM4: now also P1.1; no longer P2.2
- net SHUNT: now reaches R1.1, U1.8 (GND)
Other:
- moved on the sheet: P1, P2

Commit message: buenas noches alfred
Connections:
- net OUTM1: now also P2.2; no longer P2.1
- net OUTM2: now also P2.1; no longer P2.2
Changed lines of the file:
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@@
 	(symbol
 		(lib_id "282837-2:282837-2")
-		(at 182.88 53.34 0)
+		(at 182.88 55.88 0)
+		(mirror x)
 		(unit 1)
 		(exclude_from_sim no)
@@
 		(dnp no)
 		(property "Reference" "P2"
-			(at 186.69 53.3399 0)
+			(at 186.69 55.8801 0)
 			(effects
 				(font
@@
 		)
 		(property "Value" "282837-2"
-			(at 186.69 55.8799 0)
+			(at 186.69 53.3401 0)
 			(effects
 				(font
@@
 		)
 		(property "Footprint" "282837-2:TE_282837-2"
-			(at 182.88 53.34 0)
+			(at 182.88 55.88 0)
 			(effects
 				(font
@@
 		)
 		(property "Datasheet" ""
-			(at 182.88 53.34 0)
+			(at 182.88 55.88 0)
 			(effects
 				(font
@@
 		)
 		(property "Description" ""
-			(at 182.88 53.34 0)
+			(at 182.88 55.88 0)
 			(effects
 				(font
@@
 		)
 		(property "Comment" "282837-2"
-			(at 182.88 53.34 0)
+			(at 182.88 55.88 0)
 			(effects
 				(font
@@
 		)
 		(property "MF" "TE Connectivity"
-			(at 182.88 53.34 0)
+			(at 182.88 55.88 0)
 			(effects
 				(font
@@
 		)
 		(property "DESCRIPTION" "TERMINAL BLOCK 3.5MM 2POS PCB"
-			(at 182.88 53.34 0)
+			(at 182.88 55.88 0)
 			(effects
 				(font
@@
 		)
 		(property "PACKAGE" "None"
-			(at 182.88 53.34 0)
+			(at 182.88 55.88 0)
 			(effects
 				(font
@@
 		)
 		(property "PRICE" "0.28 USD"
-			(at 182.88 53.34 0)
+			(at 182.88 55.88 0)
 			(effects
 				(font
@@
 		)
 		(property "Package" "None"
-			(at 182.88 53.34 0)
+			(at 182.88 55.88 0)
 			(effects
 				(font
@@
 		)
 		(property "Check_prices" "https://www.snapeda.com/parts/282837-2/TE+Connectivity+AMP+Connectors/view-part/?ref=eda"
-			(at 182.88 53.34 0)
+			(at 182.88 55.88 0)
 			(effects
 				(font
@@
 		)
 		(property "Price" "None"
-			(at 182.88 53.34 0)
+			(at 182.88 55.88 0)
 			(effects
 				(font
@@
 		)
 		(property "PARTREV" "G3"
-			(at 182.88 53.34 0)
+			(at 182.88 55.88 0)
 			(effects
 				(font
@@
 		)
 		(property "SnapEDA_Link" "https://www.snapeda.com/parts/282837-2/TE+Connectivity+AMP+Connectors/view-part/?ref=snap"
-			(at 182.88 53.34 0)
+			(at 182.88 55.88 0)
 			(effects
 				(font
@@
 		)
 		(property "MP" "282837-2"
-			(at 182.88 53.34 0)
+			(at 182.88 55.88 0)
 			(effects
 				(font
@@
 		)
 		(property "Availability" "In Stock"
-			(at 182.88 53.34 0)
+			(at 182.88 55.88 0)
 			(effects
 				(font
@@
 		)
 		(property "AVAILABILITY" "Good"
-			(at 182.88 53.34 0)
+			(at 182.88 55.88 0)
 			(effects
 				(font
@@
 		)
 		(property "Description_1" "Terminal Block Connector Wire Receptacle 2 5.08 mm 30-16 AWG Green 13.5 A 250 V | TE Connectivity 282837-2"
-			(at 182.88 53.34 0)
+			(at 182.88 55.88 0)
 			(effects
 				(font

Commit message: regles de disseny i més coses
Connections:
- net REALIMENTACION_NOINV: now reaches R2.2, R3.2, U3.2 (-)
- net OUTSHUNT: now reaches R1.2, U3.3 (+)
- net AMPLIFICADO renamed OUTNOINV
Changed lines of the file:
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@@
+		)
+	)
+	(global_label "REALIMENTACION_BUFFER"
+		(shape input)
+		(at 181.61 95.25 270)
+		(fields_autoplaced yes)
+		(effects
+			(font
+				(size 1.27 1.27)
+			)
+			(justify right)
+		)
+		(property "Intersheetrefs" "${INTERSHEET_REFS}"
+			(at 181.61 122.0629 90)
+			(effects
+				(font
+					(size 1.27 1.27)
+				)
+				(justify right)
+				(hide yes)
+			)
+		)
+	)
+	(global_label "OUTSHUNT"
+		(shape input)
+		(at 129.54 85.09 270)
+		(fields_autoplaced yes)
+		(effects
+			(font
+				(size 1.27 1.27)
+			)
+			(justify right)
+		)
+		(property "Intersheetrefs" "${INTERSHEET_REFS}"
+			(at 129.54 97.8724 90)
+			(effects
+				(font
+					(size 1.27 1.27)
+				)
+				(justify right)
+				(hide yes)
+			)
 		)
 	)
@@
 		)
 	)
+	(global_label "REALIMENTACION_NOINV"
+		(shape input)
+		(at 151.13 96.52 270)
+		(fields_autoplaced yes)
+		(effects
+			(font
+				(size 1.27 1.27)
+			)
+			(justify right)
+		)
+		(property "Intersheetrefs" "${INTERSHEET_REFS}"
+			(at 151.13 121.8211 90)
+			(effects
+				(font
+					(size 1.27 1.27)
+				)
+				(justify right)
+				(hide yes)
+			)
+		)
+	)
 	(global_label "SHUNT"
 		(shape input)
@@
 		)
 	)
-	(global_label "AMPLIFICADO"
+	(global_label "OUTNOINV"
 		(shape input)
 		(at 173.99 85.09 270)
@@
 		)
 		(property "Intersheetrefs" "${INTERSHEET_REFS}"
-			(at 173.99 100.1706 90)
+			(at 173.99 97.3887 90)
 			(effects
 				(font

Commit message: hola alfred
Parts:
- P1, P2: DESCRIPTION TERMINAL BLOCK 3.5MM 2POS PCB -> (none)

Commit message: algunes millores
Parts:
- added TP5: TestPoint, TestPoint:TestPoint_Pad_1.5x1.5mm, symbol Connector:TestPoint
Connections:
- net GND: now also TP5.1
Other:
- note added: "Driver de Motor"
- moved on the sheet: C1, C2, C22, C23, C24, C25, C3, C4, C5, C6, D1, D10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

Commit message: faltan tests points
Parts:
- removed TP5: TestPoint, TestPoint:TestPoint_Pad_1.5x1.5mm, symbol Connector:TestPoint
- C25, C6: footprint Capacitor_SMD:C_1206_3216Metric -> Capacitor_SMD:C_0603_1608Metric
Changed lines of the file:
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@@
 	)
 	(junction
-		(at 114.3 96.52)
-		(diameter 0)
-		(color 0 0 0 0)
-	)
-	(junction
 		(at 231.14 132.08)
 		(diameter 0)
@@
 	(wire
 		(pts
-			(xy 114.3 96.52) (xy 121.92 96.52)
-		)
-		(stroke
-			(width 0)
-			(type default)
-		)
-	)
-	(wire
-		(pts
 			(xy 111.76 148.59) (xy 111.76 151.13)
 		)
@@
 	(wire
 		(pts
-			(xy 109.22 96.52) (xy 114.3 96.52)
+			(xy 109.22 96.52) (xy 121.92 96.52)
 		)
 		(stroke
@@
 			)
 		)
-		(property "Footprint" "Capacitor_SMD:C_1206_3216Metric"
+		(property "Footprint" "Capacitor_SMD:C_0603_1608Metric"
 			(at 201.93 76.5048 0)
 			(hide yes)
@@
 			)
 		)
-		(property "Footprint" "Capacitor_SMD:C_1206_3216Metric"
+		(property "Footprint" "Capacitor_SMD:C_0603_1608Metric"
 			(at 118.11 28.2448 0)
 			(hide yes)
@@
 					(unit 1)
 				)
-			)
-		)
-	)
-	(symbol
-		(lib_id "Connector:TestPoint")
-		(at 114.3 96.52 180)
-		(unit 1)
-		(body_style 1)
-		(exclude_from_sim no)
-		(in_bom yes)
-		(on_board yes)
-		(in_pos_files yes)
-		(dnp no)
-		(fields_autoplaced yes)
-		(property "Reference" "TP5"
-			(at 116.84 98.5519 0)
-			(show_name no)
-			(do_not_autoplace no)
-			(effects
-				(font
-					(size 1.27 1.27)
-				)
-				(justify right)
-			)
-		)
-		(property "Value" "TestPoint"
-			(at 116.84 101.0919 0)
-			(show_name no)
-			(do_not_autoplace no)
-			(effects
-				(font
-					(size 1.27 1.27)
-				)
-				(justify right)
-			)
-		)
-		(property "Footprint" "TestPoint:TestPoint_Pad_1.5x1.5mm"
-			(at 109.22 96.52 0)
-			(hide yes)
-			(show_name no)
-			(do_not_autoplace no)
-			(effects
-				(font
-					(size 1.27 1.27)
-				)
-			)
-		)
-		(property "Datasheet" ""
-			(at 109.22 96.52 0)
-			(hide yes)
-			(show_name no)
-			(do_not_autoplace no)
-			(effects
-				(font
-					(size 1.27 1.27)
-				)
-			)
-		)
-		(property "Description" "test point"
-			(at 114.3 96.52 0)
-			(hide yes)
-			(show_name no)
-			(do_not_autoplace no)
-			(effects
-				(font
-					(size 1.27 1.27)
-				)
-			)
-		)
-		(pin "1"
-		)
-		(instances
-			(project "requena.abanto_projecte_vidres"
-				(path "/4006572a-320d-4ed7-bf52-f860e1c069c6/0b0d2692-6fb2-4ddb-9a32-8981b2e43675"
-					(reference "TP5")
-					(unit 1)
-				)

Commit message: alfred butanero
Parts:
- added TP4, TP5: TestPoint_2Pole, symbol Connector:TestPoint_2Pole
Connections:
- net GND: now also TP4.2
- net GNDPWR: now also TP5.1
- net V_BAT: now also TP5.2
- net V_OUT_DCDC: now also TP4.1

Commit message: xd
Parts:
- added INA1, INB1, OUTSHUNT1, PWM1: TestPoint_2Pole, TestPoint:TestPoint_2Pads_Pitch2.54mm_Drill0.8mm, symbol Connector:TestPoint_2Pole
- R1: value 50m -> 25m
- VBAT1: renamed from TP5; footprint (none) -> TestPoint:TestPoint_2Pads_Pitch2.54mm_Drill0.8mm
- V_OUT_DCDC1: renamed from TP4; footprint (none) -> TestPoint:TestPoint_2Pads_Pitch2.54mm_Drill0.8mm
Connections:
- net GND: now also INA1.2, INB1.2, OUTSHUNT1.2, PWM1.2
- net INA: now also INA1.1
- net INB: now also INB1.1
- net OUTSHUNT: now also OUTSHUNT1.1
- net PWM: now also PWM1.1
Other:
- note added: "ETAPA DE ALIMENTACIO"
