File: KiCad/requena.abanto_projecte_vidres/requena.abanto_projecte_vidres.kicad_sch (KiCad schematic)
At the start: 0 parts

Commit message: Creacio d'etapes
Other:
- added sheet Etapa_de_alimentacio (Etapa_de_alimentacio.kicad_sch)
- added sheet Etapa_de_comunicacio (Etapa_de_comunicacio.kicad_sch)
- added sheet Etapa_de_processament (Etapa_de_processament.kicad_sch)
- added sheet Etapa_de_sensors (Etapa_de_sensors.kicad_sch)
- added sheet etapa_de_potencia (etapa_de_potencia.kicad_sch)
- note added: "Etapa de alimentació"
- note added: "Etapa de comuniació"
- note added: "Etapa de potència"
- note added: "Etapa de processament"
- note added: "Etapa de sensors"

Commit message: Millora projecte 1
Other:
- removed sheet Etapa_de_alimentacio
- note removed: "Etapa de alimentació"
Changed lines of the file:
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@@
-		)
-	)
-	(text "Etapa de alimentació"
-		(exclude_from_sim no)
-		(at 61.468 19.812 0)
-		(effects
-			(font
-				(size 5 5)
-			)
 		)
 	)
@@
 			)
 		)
-	)
-	(sheet
-		(at 17.78 13.97)
-		(size 90.17 41.91)
-		(exclude_from_sim no)
-		(in_bom yes)
-		(on_board yes)
-		(dnp no)
-		(fields_autoplaced yes)
-		(stroke
-			(width 0.1524)
-			(type solid)
-		)
-		(fill
-			(color 0 0 0 0.0000)
-		)
-		(property "Sheetname" "Etapa_de_alimentacio"
-			(at 17.78 13.2584 0)
-			(effects
-				(font
-					(size 1.27 1.27)
-				)
-				(justify left bottom)
-			)
-		)
-		(property "Sheetfile" "Etapa_de_alimentacio.kicad_sch"
-			(at 17.78 56.4646 0)
-			(effects
-				(font
-					(size 1.27 1.27)
-				)
-				(justify left top)
-			)
-		)
-		(instances
-			(project "requena.abanto_projecte_vidres"
-				(path "/4006572a-320d-4ed7-bf52-f860e1c069c6"
-					(page "3")
-				)
-			)
-		)

Commit message: guardado
Other:
- removed sheet Etapa_de_comunicacio
- removed sheet Etapa_de_sensors
- note removed: "Etapa de comuniació"
- note removed: "Etapa de sensors"
Changed lines of the file:
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@@
 	(text "Etapa de processament\n"
 		(exclude_from_sim no)
-		(at 244.094 19.304 0)
+		(at 165.354 54.864 0)
 		(effects
 			(font
@@
 		)
 	)
-	(text "Etapa de comuniació\n"
-		(exclude_from_sim no)
-		(at 60.198 68.326 0)
-		(effects
-			(font
-				(size 5 5)
-			)
-		)
-	)
-	(text "Etapa de sensors \n\n"
-		(exclude_from_sim no)
-		(at 148.844 72.39 0)
-		(effects
-			(font
-				(size 5 5)
-			)
-		)
-	)
 	(text "Etapa de potència "
 		(exclude_from_sim no)
-		(at 154.686 19.558 0)
+		(at 75.946 55.118 0)
 		(effects
 			(font
@@
 	)
 	(sheet
-		(at 111.76 13.97)
+		(at 33.02 49.53)
 		(size 90.17 41.91)
 		(exclude_from_sim no)
@@
 		)
 		(property "Sheetname" "etapa_de_potencia"
-			(at 111.76 13.2584 0)
+			(at 33.02 48.8184 0)
 			(effects
 				(font
@@
 		)
 		(property "Sheetfile" "etapa_de_potencia.kicad_sch"
-			(at 111.76 56.4646 0)
+			(at 33.02 92.0246 0)
 			(effects
 				(font
@@
 	)
 	(sheet
-		(at 17.78 62.23)
-		(size 90.17 41.91)
-		(exclude_from_sim no)
-		(in_bom yes)
-		(on_board yes)
-		(dnp no)
-		(fields_autoplaced yes)
-		(stroke
-			(width 0.1524)
-			(type solid)
-		)
-		(fill
-			(color 0 0 0 0.0000)
-		)
-		(property "Sheetname" "Etapa_de_comunicacio"
-			(at 17.78 61.5184 0)
-			(effects
-				(font
-					(size 1.27 1.27)
-				)
-				(justify left bottom)
-			)
-		)
-		(property "Sheetfile" "Etapa_de_comunicacio.kicad_sch"
-			(at 17.78 104.7246 0)
-			(effects
-				(font
-					(size 1.27 1.27)
-				)
-				(justify left top)
-			)
-		)
-		(instances
-			(project "requena.abanto_projecte_vidres"
-				(path "/4006572a-320d-4ed7-bf52-f860e1c069c6"
-					(page "5")
-				)
-			)
-		)
-	)
-	(sheet
-		(at 205.74 13.97)
+		(at 127 49.53)
 		(size 76.2 41.91)
 		(exclude_from_sim no)
@@
 		)
 		(property "Sheetname" "Etapa_de_processament"
-			(at 205.74 13.2584 0)
+			(at 127 48.8184 0)
 			(effects
 				(font
@@
 		)
 		(property "Sheetfile" "Etapa_de_processament.kicad_sch"
-			(at 205.74 56.4646 0)
+			(at 127 92.0246 0)
 			(effects
 				(font
@@
 				)
 			)
-		)
-	)
-	(sheet
-		(at 111.76 62.23)
-		(size 90.17 40.64)
-		(exclude_from_sim no)
-		(in_bom yes)
-		(on_board yes)
-		(dnp no)
-		(fields_autoplaced yes)
-		(stroke
-			(width 0.1524)
-			(type solid)
-		)
-		(fill
-			(color 0 0 0 0.0000)
-		)
-		(property "Sheetname" "Etapa_de_sensors"
-			(at 111.76 61.5184 0)
-			(effects
-				(font
-					(size 1.27 1.27)
-				)
-				(justify left bottom)
-			)
-		)
-		(property "Sheetfile" "Etapa_de_sensors.kicad_sch"
-			(at 111.76 103.4546 0)
-			(effects
-				(font
-					(size 1.27 1.27)
-				)
-				(justify left top)
-			)
-		)
-		(instances
-			(project "requena.abanto_projecte_vidres"
-				(path "/4006572a-320d-4ed7-bf52-f860e1c069c6"
-					(page "6")
-				)
-			)

Commit message: :(
Other:
- company: (none) -> AUTORS: ÀLEX REQUENA i ALFRED ABANTO
- title: (none) -> PROJECTE ALÇAVIDRES
Changed lines of the file:
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@@
 	(generator_version "9.0")
 	(paper "A4")
+	(title_block
+		(title "PROJECTE ALÇAVIDRES")
+		(company "AUTORS: ÀLEX REQUENA i ALFRED ABANTO")
+	)
 	(text "Etapa de processament\n"
 		(exclude_from_sim no)
